Commit message: description: update ur5 mounting orientation

File: rbkairos_description/robots/rbkairos_ur5.urdf.xacro (robot description, xacro)
@@ -19,5 +19,5 @@
   <xacro:property name="arm_orientation_r" value="0"/>
   <xacro:property name="arm_orientation_p" value="0"/>
-  <xacro:property name="arm_orientation_y" value="${-3*pi/4}"/>
+  <xacro:property name="arm_orientation_y" value="0.0"/>
   <xacro:macro name="rbkairos" params="prefix publish_bf hq load_kinematics_file">
 		<!-- *************** -->

File: rbkairos_description/robots/versions/rbkairos_ur5_egh.urdf.xacro (robot description, xacro)
@@ -23,5 +23,5 @@
   <xacro:property name="arm_orientation_r" value="0"/>
   <xacro:property name="arm_orientation_p" value="0"/>
-  <xacro:property name="arm_orientation_y" value="${-3*pi/4}"/>
+  <xacro:property name="arm_orientation_y" value="${pi/4}"/>
   <xacro:macro name="rbkairos" params="prefix publish_bf hq load_kinematics_file">
 		<!-- *************** -->
