Commit message: Erased box on vgc10 ur10 urdf

File: rbkairos_description/robots/rbkairos_ur10_vgc10.urdf.xacro (robot description, xacro)
@@ -5,5 +5,4 @@
   	<!-- ***************** -->
   	<!-- First we import all posible elements defined in the urdf.xacro files. All these elements are defined as macro:xacros -->
-    <xacro:include filename="$(find rbkairos_description)/urdf/structures/box.urdf.xacro" />
   	<!-- Import summit XL base elements -->
   	<xacro:include filename="$(find summit_xl_description)/urdf/bases/summit_xls_base.urdf.xacro" />
@@ -88,7 +87,4 @@
   			</joint>
   		</xacro:if>
-      <xacro:container prefix="$(arg prefix)" parent="$(arg prefix)base_link">
-        <origin xyz="1 1 0" rpy="0 0 0"/>
-      </xacro:container>
       <!-- OnRobot VGC-10 -->
       <xacro:vgc10 prefix="$(arg prefix)vgc10" parent="$(arg prefix)arm_tool0">

Commit message: Rbkairos_description: Corrected unused arg "load_kinematics_file"

File: rbkairos_description/robots/rbkairos_ur10_vgc10.urdf.xacro (robot description, xacro)
@@ -76,5 +76,5 @@
   		</xacro:omni_wheel>
       <!-- UR-10 ARM -->
-  		<xacro:if value="$(arg has_arm)">
+  		<!--xacro:if value="$(arg has_arm)">
   			<xacro:ur10_robot prefix="$(arg prefix)arm_" joint_limited="true"
   			shoulder_pan_lower_limit="${-pi}" shoulder_pan_upper_limit="${pi}"
@@ -86,5 +86,29 @@
   				<child link="$(arg prefix)arm_base_link" />
   			</joint>
-  		</xacro:if>
+  		</xacro:if-->
+      <!-- UR-10 ARM -->
+      <xacro:if value="$(arg load_kinematics_file)">
+          <xacro:ur10_robot prefix="$(arg prefix)arm_" joint_limited="true"
+          shoulder_pan_lower_limit="${-pi}" shoulder_pan_upper_limit="${pi}"
+          wrist_3_lower_limit="${-pi}" wrist_3_upper_limit="${pi}"
+          kinematics_file="${load_yaml('$(find rbkairos_control)/config/ur10_calibration.yaml')}">
+          </xacro:ur10_robot>
+          <joint name="$(arg prefix)arm_base_joint" type="fixed">
+              <origin xyz="${arm_position_x} ${arm_position_y} ${arm_position_z}" rpy="${arm_orientation_r} ${arm_orientation_p} ${arm_orientation_y}"/>
+              <parent link="$(arg prefix)base_link" />
+              <child link="$(arg prefix)arm_base_link" />
+          </joint>
+      </xacro:if>
+      <xacro:unless value="$(arg load_kinematics_file)">
+          <xacro:ur10_robot prefix="$(arg prefix)arm_" joint_limited="true"
+          shoulder_pan_lower_limit="${-pi}" shoulder_pan_upper_limit="${pi}"
+          wrist_3_lower_limit="${-pi}" wrist_3_upper_limit="${pi}">
+          </xacro:ur10_robot>
+          <joint name="$(arg prefix)arm_base_joint" type="fixed">
+          <origin xyz="${arm_position_x} ${arm_position_y} ${arm_position_z}" rpy="${arm_orientation_r} ${arm_orientation_p} ${arm_orientation_y}"/>
+          <parent link="$(arg prefix)base_link" />
+          <child link="$(arg prefix)arm_base_link" />
+          </joint>
+      </xacro:unless>
       <!-- OnRobot VGC-10 -->
       <xacro:vgc10 prefix="$(arg prefix)vgc10" parent="$(arg prefix)arm_tool0">
