Commit message: decription: Add xacro properties and the correct pos for ur5

File: rbkairos_description/robots/rbkairos_ur10.urdf.xacro (robot description, xacro)
@@ -13,6 +13,12 @@
 	<xacro:arg name="prefix" default="robot_"/>
 	<xacro:arg name="ros_planar_move_plugin" default="false"/>
-	<xacro:arg name="has_arm" default="true"/>
-  <xacro:macro name="rbkairos" params="prefix publish_bf hq">
+  <xacro:arg name="load_kinematics_file" default="false"/> <!-- Necesarry for ur_description compatible with official ur drivers-->
+  <xacro:property name="arm_position_x" value="0"/>
+  <xacro:property name="arm_position_y" value="0"/>
+  <xacro:property name="arm_position_z" value="0.38212"/>
+  <xacro:property name="arm_orientation_r" value="0"/>
+  <xacro:property name="arm_orientation_p" value="0"/>
+  <xacro:property name="arm_orientation_y" value="0"/>
+  <xacro:macro name="rbkairos" params="prefix publish_bf hq load_kinematics_file">
 		<!-- *************** -->
 		<!-- Robots Elements -->
@@ -21,16 +27,28 @@
 		<!-- RBKAIROS base -->
 		<xacro:rbkairos_base prefix="$(arg prefix)" publish_bf="true" hq="true"/>
-		<!-- UR-10 ARM -->
-		<xacro:if value="$(arg has_arm)">
-			<xacro:ur10_robot prefix="$(arg prefix)arm_" joint_limited="true"
-			shoulder_pan_lower_limit="${-pi}" shoulder_pan_upper_limit="${pi}"
-			wrist_3_lower_limit="${-pi}" wrist_3_upper_limit="${pi}">
-			</xacro:ur10_robot>
-			<joint name="$(arg prefix)arm_base_joint" type="fixed">
-				<origin xyz="0.0 0 0.38212" rpy="0 0 ${PI*0}"/>
-				<parent link="$(arg prefix)base_link" />
-				<child link="$(arg prefix)arm_base_link" />
-			</joint>
+		<!-- UR-5 ARM -->
+		<xacro:if value="$(arg load_kinematics_file)">
+        <xacro:ur10_robot prefix="$(arg prefix)arm_" joint_limited="true"
+          shoulder_pan_lower_limit="${-pi}" shoulder_pan_upper_limit="${pi}"
+          wrist_3_lower_limit="${-pi}" wrist_3_upper_limit="${pi}"
+          kinematics_file="${load_yaml('$(find rbkairos_control)/config/ur10_calibration.yaml')}">
+        </xacro:ur10_robot>
+        <joint name="$(arg prefix)arm_base_joint" type="fixed">
+          <origin xyz="${arm_position_x} ${arm_position_y} ${arm_position_z}" rpy="${arm_orientation_r} ${arm_orientation_p} ${arm_orientation_y}"/>
+          <parent link="$(arg prefix)base_link" />
+          <child link="$(arg prefix)arm_base_link" />
+        </joint>
 		</xacro:if>
+		<xacro:unless value="$(arg load_kinematics_file)">
+        <xacro:ur10_robot prefix="$(arg prefix)arm_" joint_limited="true"
+          shoulder_pan_lower_limit="${-pi}" shoulder_pan_upper_limit="${pi}"
+          wrist_3_lower_limit="${-pi}" wrist_3_upper_limit="${pi}">
+        </xacro:ur10_robot>
+        <joint name="$(arg prefix)arm_base_joint" type="fixed">
+          <origin xyz="${arm_position_x} ${arm_position_y} ${arm_position_z}" rpy="${arm_orientation_r} ${arm_orientation_p} ${arm_orientation_y}"/>
+          <parent link="$(arg prefix)base_link" />
+          <child link="$(arg prefix)arm_base_link" />
+        </joint>
+		</xacro:unless>
 	</xacro:macro>
    <!-- Gazebo ros control pluggins -->
@@ -39,4 +57,4 @@
 	   <xacro:omni_steering prefix="$(arg prefix)" publish_tf="false"/>
    </xacro:if>
-   <xacro:rbkairos prefix="$(arg prefix)" publish_bf="true" hq="true"/>
+   <xacro:rbkairos prefix="$(arg prefix)" publish_bf="true" hq="true" load_kinematics_file="$(arg load_kinematics_file)"/>
 </robot>

File: rbkairos_description/robots/rbkairos_ur5.urdf.xacro (robot description, xacro)
@@ -13,6 +13,12 @@
 	<xacro:arg name="prefix" default="robot_"/>
 	<xacro:arg name="ros_planar_move_plugin" default="false"/>
-	<xacro:arg name="has_arm" default="true"/>
-  <xacro:macro name="rbkairos" params="prefix publish_bf hq">
+	<xacro:arg name="load_kinematics_file" default="false"/> <!-- Necesarry for ur_description compatible with official ur drivers-->
+  <xacro:property name="arm_position_x" value="0.1883"/>
+  <xacro:property name="arm_position_y" value="0"/>
+  <xacro:property name="arm_position_z" value="0.38212"/>
+  <xacro:property name="arm_orientation_r" value="0"/>
+  <xacro:property name="arm_orientation_p" value="0"/>
+  <xacro:property name="arm_orientation_y" value="${-3*pi/4}"/>
+  <xacro:macro name="rbkairos" params="prefix publish_bf hq load_kinematics_file">
 		<!-- *************** -->
 		<!-- Robots Elements -->
@@ -22,15 +28,27 @@
 		<xacro:rbkairos_base prefix="$(arg prefix)" publish_bf="true" hq="true"/>
 		<!-- UR-5 ARM -->
-		<xacro:if value="$(arg has_arm)">
-            <xacro:ur5_robot prefix="$(arg prefix)arm_" joint_limited="true"
-                shoulder_pan_lower_limit="${-pi}" shoulder_pan_upper_limit="${pi}"
-                wrist_3_lower_limit="${-pi}" wrist_3_upper_limit="${pi}">
-            </xacro:ur5_robot>
-            <joint name="$(arg prefix)arm_base_joint" type="fixed">
-				<origin xyz="0.0 0 0.38212" rpy="0 0 ${PI*0}"/>
-				<parent link="$(arg prefix)base_link" />
-				<child link="$(arg prefix)arm_base_link" />
-			</joint>
+		<xacro:if value="$(arg load_kinematics_file)">
+        <xacro:ur5_robot prefix="$(arg prefix)arm_" joint_limited="true"
+          shoulder_pan_lower_limit="${-pi}" shoulder_pan_upper_limit="${pi}"
+          wrist_3_lower_limit="${-pi}" wrist_3_upper_limit="${pi}"
+          kinematics_file="${load_yaml('$(find rbkairos_control)/config/ur5_calibration.yaml')}">
+        </xacro:ur5_robot>
+        <joint name="$(arg prefix)arm_base_joint" type="fixed">
+          <origin xyz="${arm_position_x} ${arm_position_y} ${arm_position_z}" rpy="${arm_orientation_r} ${arm_orientation_p} ${arm_orientation_y}"/>
+          <parent link="$(arg prefix)base_link" />
+          <child link="$(arg prefix)arm_base_link" />
+        </joint>
 		</xacro:if>
+		<xacro:unless value="$(arg load_kinematics_file)">
+        <xacro:ur5_robot prefix="$(arg prefix)arm_" joint_limited="true"
+          shoulder_pan_lower_limit="${-pi}" shoulder_pan_upper_limit="${pi}"
+          wrist_3_lower_limit="${-pi}" wrist_3_upper_limit="${pi}">
+        </xacro:ur5_robot>
+        <joint name="$(arg prefix)arm_base_joint" type="fixed">
+          <origin xyz="${arm_position_x} ${arm_position_y} ${arm_position_z}" rpy="${arm_orientation_r} ${arm_orientation_p} ${arm_orientation_y}"/>
+          <parent link="$(arg prefix)base_link" />
+          <child link="$(arg prefix)arm_base_link" />
+        </joint>
+		</xacro:unless>
 	</xacro:macro>
    <!-- Gazebo ros control pluggins -->
@@ -39,4 +57,4 @@
 	   <xacro:omni_steering prefix="$(arg prefix)" publish_tf="false"/>
    </xacro:if>
-   <xacro:rbkairos prefix="$(arg prefix)" publish_bf="true" hq="true"/>
+   <xacro:rbkairos prefix="$(arg prefix)" publish_bf="true" hq="true" load_kinematics_file="$(arg load_kinematics_file)"/>
 </robot>

File: rbkairos_description/robots/versions/rbkairos_ur5_egh.urdf.xacro (robot description, xacro)
@@ -9,13 +9,20 @@
 	<!-- Include UR-5 ARM -->
 	<xacro:include filename="$(find ur_description)/urdf/ur5.urdf.xacro" />
-    <!-- Include EGH TODO -->
-    <!-- Import all available sensors -->
-  	<xacro:include filename="$(find robotnik_sensors)/urdf/all_sensors.urdf.xacro" />
+  <!-- Include EGH TODO -->
+	<xacro:include filename="$(find egh_gripper_description)/urdf/egh_gripper.urdf.xacro" />
+  <!-- Import all available sensors -->
+  <xacro:include filename="$(find robotnik_sensors)/urdf/all_sensors.urdf.xacro" />
 	<!-- Flag to select the high or low quality model -->
 	<xacro:property name="hq" value="true" />
 	<xacro:arg name="prefix" default="robot_"/>
 	<xacro:arg name="ros_planar_move_plugin" default="false"/>
-	<xacro:arg name="has_arm" default="true"/>
-  <xacro:macro name="rbkairos" params="prefix publish_bf hq">
+	<xacro:arg name="load_kinematics_file" default="false"/> <!-- Necesarry for ur_description compatible with official ur drivers-->
+  <xacro:property name="arm_position_x" value="0.1883"/>
+  <xacro:property name="arm_position_y" value="0"/>
+  <xacro:property name="arm_position_z" value="0.38212"/>
+  <xacro:property name="arm_orientation_r" value="0"/>
+  <xacro:property name="arm_orientation_p" value="0"/>
+  <xacro:property name="arm_orientation_y" value="${-3*pi/4}"/>
+  <xacro:macro name="rbkairos" params="prefix publish_bf hq load_kinematics_file">
 		<!-- *************** -->
 		<!-- Robots Elements -->
@@ -25,23 +32,35 @@
 		<xacro:rbkairos_base prefix="$(arg prefix)" publish_bf="true" hq="true"/>
 		<!-- UR-5 ARM -->
-		<xacro:if value="$(arg has_arm)">
-            <xacro:ur5_robot prefix="$(arg prefix)arm_" joint_limited="true"
-                shoulder_pan_lower_limit="${-pi}" shoulder_pan_upper_limit="${pi}"
-                wrist_3_lower_limit="${-pi}" wrist_3_upper_limit="${pi}">
-            </xacro:ur5_robot>
-            <joint name="$(arg prefix)arm_base_joint" type="fixed">
-				<origin xyz="0.0 0 0.38212" rpy="0 0 ${PI*0}"/>
-				<parent link="$(arg prefix)base_link" />
-				<child link="$(arg prefix)arm_base_link" />
-			</joint>
+		<xacro:if value="$(arg load_kinematics_file)">
+        <xacro:ur5_robot prefix="$(arg prefix)arm_" joint_limited="true"
+          shoulder_pan_lower_limit="${-pi}" shoulder_pan_upper_limit="${pi}"
+          wrist_3_lower_limit="${-pi}" wrist_3_upper_limit="${pi}"
+          kinematics_file="${load_yaml('$(find rbkairos_control)/config/ur5_calibration.yaml')}">
+        </xacro:ur5_robot>
+        <joint name="$(arg prefix)arm_base_joint" type="fixed">
+          <origin xyz="${arm_position_x} ${arm_position_y} ${arm_position_z}" rpy="${arm_orientation_r} ${arm_orientation_p} ${arm_orientation_y}"/>
+          <parent link="$(arg prefix)base_link" />
+          <child link="$(arg prefix)arm_base_link" />
+        </joint>
 		</xacro:if>
-		<!-- Schunk EGH TODO -->
-		<!--xacro:egh_xacro name="$(arg prefix)egh" parent="$(arg prefix)arm_tool0" finger_length="0.023" finger_tip="0">
-			<origin xyz="0.0 0.0 0.0" rpy="0 0 0"/>
-		</xacro:egh_xacro-->
+		<xacro:unless value="$(arg load_kinematics_file)">
+        <xacro:ur5_robot prefix="$(arg prefix)arm_" joint_limited="true"
+          shoulder_pan_lower_limit="${-pi}" shoulder_pan_upper_limit="${pi}"
+          wrist_3_lower_limit="${-pi}" wrist_3_upper_limit="${pi}">
+        </xacro:ur5_robot>
+        <joint name="$(arg prefix)arm_base_joint" type="fixed">
+          <origin xyz="${arm_position_x} ${arm_position_y} ${arm_position_z}" rpy="${arm_orientation_r} ${arm_orientation_p} ${arm_orientation_y}"/>
+          <parent link="$(arg prefix)base_link" />
+          <child link="$(arg prefix)arm_base_link" />
+        </joint>
+		</xacro:unless>
+		<!-- Schunk EGH -->
+		<xacro:egh_gripper prefix="$(arg prefix)egh_gripper" parent="$(arg prefix)arm_tool0">
+			<origin xyz="0.0 0.0 0.0" rpy="0 -${pi/2} 0"/>
+		</xacro:egh_gripper>
         <!-- Intel Realsense -->
-        <xacro:sensor_r430 prefix="$(arg prefix)arm_rgbd_camera" parent="$(arg prefix)arm_tool0" prefix_topic="front_rgbd_camera">
-  			<origin xyz="0.0 -0.05 -0.01" rpy="${pi/2} ${-pi/2} 0"/>
-  		</xacro:sensor_r430>
+    <xacro:sensor_r430 prefix="$(arg prefix)arm_rgbd_camera" parent="$(arg prefix)arm_tool0" prefix_topic="front_rgbd_camera">
+      <origin xyz="0.0 -0.05 -0.01" rpy="${pi/2} ${-pi/2} 0"/>
+    </xacro:sensor_r430>
 	</xacro:macro>
    <!-- Gazebo ros control pluggins -->
@@ -50,4 +69,4 @@
 	   <xacro:omni_steering prefix="$(arg prefix)" publish_tf="false"/>
    </xacro:if>
-   <xacro:rbkairos prefix="$(arg prefix)" publish_bf="true" hq="true"/>
+   <xacro:rbkairos prefix="$(arg prefix)" publish_bf="true" hq="true" load_kinematics_file="$(arg load_kinematics_file)"/>
 </robot>

Commit message: rbkairos_description: Update rbkairos_ur10 urdf to no load rbkairos_base macro

File: rbkairos_description/robots/rbkairos_ur10.urdf.xacro (robot description, xacro)
@@ -1,60 +1,121 @@
 <?xml version="1.0"?>
 <robot name="rbkairos" xmlns:xacro="http://wiki.ros.org/xacro">
-	<!-- ***************** -->
-	<!-- Imported elements -->
-	<!-- ***************** -->
-	<!-- First we import all posible elements defined in the urdf.xacro files. All these elements are defined as macro:xacros -->
-	<!-- Import summit XL base elements -->
-	<xacro:include filename="$(find rbkairos_description)/urdf/bases/rbkairos_base.urdf.xacro" />
-	<!-- Include UR-10 ARM -->
+  	<!-- ***************** -->
+  	<!-- Imported elements -->
+  	<!-- ***************** -->
+  	<!-- First we import all posible elements defined in the urdf.xacro files. All these elements are defined as macro:xacros -->
+  	<!-- Import summit XL base elements -->
+  	<xacro:include filename="$(find summit_xl_description)/urdf/bases/summit_xls_base.urdf.xacro" />
+    <!-- Include UR-10 ARM -->
 	<xacro:include filename="$(find ur_description)/urdf/ur10.urdf.xacro" />
-	<!-- Flag to select the high or low quality model -->
-	<xacro:property name="hq" value="true" />
-	<xacro:arg name="prefix" default="robot_"/>
-	<xacro:arg name="ros_planar_move_plugin" default="false"/>
-  <xacro:arg name="load_kinematics_file" default="false"/> <!-- Necesarry for ur_description compatible with official ur drivers-->
-  <xacro:property name="arm_position_x" value="0"/>
-  <xacro:property name="arm_position_y" value="0"/>
-  <xacro:property name="arm_position_z" value="0.38212"/>
-  <xacro:property name="arm_orientation_r" value="0"/>
-  <xacro:property name="arm_orientation_p" value="0"/>
-  <xacro:property name="arm_orientation_y" value="0"/>
-  <xacro:macro name="rbkairos" params="prefix publish_bf hq load_kinematics_file">
-		<!-- *************** -->
-		<!-- Robots Elements -->
-		<!-- *************** -->
-		<!-- Here we create the robot elements using the xacro:macros imported at the beggining of this file -->
-		<!-- RBKAIROS base -->
-		<xacro:rbkairos_base prefix="$(arg prefix)" publish_bf="true" hq="true"/>
-		<!-- UR-5 ARM -->
+  	<!-- Import summit XL wheels -->
+  	<xacro:include filename="$(find summit_xl_description)/urdf/wheels/omni_wheel.urdf.xacro" />
+  	<xacro:include filename="$(find summit_xl_description)/urdf/wheels/rubber_wheel.urdf.xacro" />
+  	<xacro:include filename="$(find summit_xl_description)/urdf/structures/structure_hokuyo.urdf.xacro" />
+  	<!-- Import all available sensors -->
+  	<xacro:include filename="$(find robotnik_sensors)/urdf/all_sensors.urdf.xacro" />
+  	<xacro:property name="PI" value="3.1415926535897931"/>
+  	<!-- Wheel parameters -->
+  	<xacro:property name="wheel_offset_x" value="0.2225" />    <!-- x,y,z in translation from base_link to the center of the wheel -->
+  	<xacro:property name="wheel_offset_y" value="0.2045" />
+  	<xacro:property name="wheel_offset_z" value="0.0" />
+  	<xacro:property name="front_laser_offset_x" value="0.2865"/>
+  	<xacro:property name="front_laser_offset_y" value="-0.20894"/>
+  	<xacro:property name="front_laser_offset_z" value="0.2973"/>
+  	<xacro:property name="rear_laser_offset_x" value="-0.2865"/>
+  	<xacro:property name="rear_laser_offset_y" value="0.20894"/>
+  	<xacro:property name="rear_laser_offset_z" value="0.2973"/>
+  	<xacro:property name="front_ptz_camera_offset_x" value="0.308"/>
+  	<xacro:property name="front_ptz_camera_offset_y" value="0.141"/>
+  	<xacro:property name="front_ptz_camera_offset_z" value="0.195"/>
+  	<xacro:property name="rear_ptz_camera_offset_x" value="-0.308"/>
+  	<xacro:property name="rear_ptz_camera_offset_y" value="-0.141"/>
+  	<xacro:property name="rear_ptz_camera_offset_z" value="0.195"/>
+    <xacro:property name="imu_offset_x" value="0.127"/>
+  	<xacro:property name="imu_offset_y" value="-0.129"/>
+  	<xacro:property name="imu_offset_z" value="0.212"/>
+  	<xacro:property name="front_rgbd_camera_offset_x" value="0.35850"/>
+  	<xacro:property name="front_rgbd_camera_offset_y" value="0.0"/>
+  	<xacro:property name="front_rgbd_camera_offset_z" value="0.25062"/>
+  	<xacro:property name="gps_offset_x" value="-0.365"/>
+  	<xacro:property name="gps_offset_y" value="-0.167"/>
+  	<xacro:property name="gps_offset_z" value="0.302"/>
+  	<!-- Flag to select the high or low quality model -->
+  	<xacro:property name="hq" value="true" />
+  	<xacro:arg name="prefix" default="robot_"/>
+  	<xacro:arg name="ros_planar_move_plugin" default="false"/>
+    <xacro:arg name="load_kinematics_file" default="false"/> <!-- Necesarry for ur_description compatible with official ur drivers-->
+    <xacro:property name="arm_position_x" value="0.0"/>
+    <xacro:property name="arm_position_y" value="0"/>
+    <xacro:property name="arm_position_z" value="0.383612"/>
+    <xacro:property name="arm_orientation_r" value="0"/>
+    <xacro:property name="arm_orientation_p" value="0"/>
+    <xacro:property name="arm_orientation_y" value="0"/>
+    <xacro:macro name="rbkairos" params="prefix publish_bf hq load_kinematics_file">
+  		<!-- *************** -->
+  		<!-- Robots Elements -->
+  		<!-- *************** -->
+  		<!-- Here we create the robot elements using the xacro:macros imported at the beggining of this file -->
+  		<!-- Summit XL base -->
+  		<xacro:summit_xls_base prefix="$(arg prefix)" publish_bf="true" hq="${hq}" />
+  		<xacro:omni_wheel prefix="$(arg prefix)front_right" parent="$(arg prefix)base_link" reflect="false" hq="${hq}">
+  			<origin xyz="${wheel_offset_x} -${wheel_offset_y} ${wheel_offset_z}" rpy="0 0 0"/>
+  		</xacro:omni_wheel>
+  		<xacro:omni_wheel prefix="$(arg prefix)front_left" parent="$(arg prefix)base_link" reflect="true" hq="${hq}">
+  			<origin xyz="${wheel_offset_x} ${wheel_offset_y} ${wheel_offset_z}" rpy="0 0 0"/>
+  		</xacro:omni_wheel>
+  		<xacro:omni_wheel prefix="$(arg prefix)back_left" parent="$(arg prefix)base_link" reflect="true" hq="${hq}">
+  			<origin xyz="-${wheel_offset_x} ${wheel_offset_y} ${wheel_offset_z}" rpy="0 0 0"/>
+  		</xacro:omni_wheel>
+  		<xacro:omni_wheel prefix="$(arg prefix)back_right" parent="$(arg prefix)base_link" reflect="false" hq="${hq}">
+  			<origin xyz="-${wheel_offset_x} -${wheel_offset_y} ${wheel_offset_z}" rpy="0 0 0"/>
+  		</xacro:omni_wheel>
+        <!-- UR-10 ARM -->
 		<xacro:if value="$(arg load_kinematics_file)">
-        <xacro:ur10_robot prefix="$(arg prefix)arm_" joint_limited="true"
-          shoulder_pan_lower_limit="${-pi}" shoulder_pan_upper_limit="${pi}"
-          wrist_3_lower_limit="${-pi}" wrist_3_upper_limit="${pi}"
-          kinematics_file="${load_yaml('$(find rbkairos_control)/config/ur10_calibration.yaml')}">
-        </xacro:ur10_robot>
-        <joint name="$(arg prefix)arm_base_joint" type="fixed">
-          <origin xyz="${arm_position_x} ${arm_position_y} ${arm_position_z}" rpy="${arm_orientation_r} ${arm_orientation_p} ${arm_orientation_y}"/>
-          <parent link="$(arg prefix)base_link" />
-          <child link="$(arg prefix)arm_base_link" />
-        </joint>
+            <xacro:ur10_robot prefix="$(arg prefix)arm_" joint_limited="true"
+            shoulder_pan_lower_limit="${-pi}" shoulder_pan_upper_limit="${pi}"
+            wrist_3_lower_limit="${-pi}" wrist_3_upper_limit="${pi}"
+            kinematics_file="${load_yaml('$(find rbkairos_control)/config/ur10_calibration.yaml')}">
+            </xacro:ur10_robot>
+            <joint name="$(arg prefix)arm_base_joint" type="fixed">
+                <origin xyz="${arm_position_x} ${arm_position_y} ${arm_position_z}" rpy="${arm_orientation_r} ${arm_orientation_p} ${arm_orientation_y}"/>
+                <parent link="$(arg prefix)base_link" />
+                <child link="$(arg prefix)arm_base_link" />
+            </joint>
 		</xacro:if>
 		<xacro:unless value="$(arg load_kinematics_file)">
-        <xacro:ur10_robot prefix="$(arg prefix)arm_" joint_limited="true"
-          shoulder_pan_lower_limit="${-pi}" shoulder_pan_upper_limit="${pi}"
-          wrist_3_lower_limit="${-pi}" wrist_3_upper_limit="${pi}">
-        </xacro:ur10_robot>
-        <joint name="$(arg prefix)arm_base_joint" type="fixed">
-          <origin xyz="${arm_position_x} ${arm_position_y} ${arm_position_z}" rpy="${arm_orientation_r} ${arm_orientation_p} ${arm_orientation_y}"/>
-          <parent link="$(arg prefix)base_link" />
-          <child link="$(arg prefix)arm_base_link" />
-        </joint>
+            <xacro:ur10_robot prefix="$(arg prefix)arm_" joint_limited="true"
+            shoulder_pan_lower_limit="${-pi}" shoulder_pan_upper_limit="${pi}"
+            wrist_3_lower_limit="${-pi}" wrist_3_upper_limit="${pi}">
+            </xacro:ur10_robot>
+            <joint name="$(arg prefix)arm_base_joint" type="fixed">
+            <origin xyz="${arm_position_x} ${arm_position_y} ${arm_position_z}" rpy="${arm_orientation_r} ${arm_orientation_p} ${arm_orientation_y}"/>
+            <parent link="$(arg prefix)base_link" />
+            <child link="$(arg prefix)arm_base_link" />
+            </joint>
 		</xacro:unless>
-	</xacro:macro>
-   <!-- Gazebo ros control pluggins -->
-   <xacro:ros_control/>
-   <xacro:if value="$(arg ros_planar_move_plugin)">
-	   <xacro:omni_steering prefix="$(arg prefix)" publish_tf="false"/>
-   </xacro:if>
-   <xacro:rbkairos prefix="$(arg prefix)" publish_bf="true" hq="true" load_kinematics_file="$(arg load_kinematics_file)"/>
+        <!-- IMU -->
+  		<xacro:sensor_imu_hector prefix="$(arg prefix)imu" parent="$(arg prefix)base_link">
+  			<origin xyz="${imu_offset_x} ${imu_offset_y} ${imu_offset_z}" rpy="0 0 0"/>
+  		</xacro:sensor_imu_hector>
+  		<!-- SENSORS -->
+  		<xacro:sensor_sick_s300 prefix="$(arg prefix)front_laser" parent="$(arg prefix)base_link" prefix_topic="front_laser">
+  			<origin xyz="${front_laser_offset_x} ${front_laser_offset_y} ${front_laser_offset_z}" rpy="0 ${-PI} ${3/4*PI}" />
+  		</xacro:sensor_sick_s300>
+  		<xacro:sensor_sick_s300 prefix="$(arg prefix)rear_laser" parent="$(arg prefix)base_link" prefix_topic="rear_laser">
+  			<origin xyz="${rear_laser_offset_x} ${rear_laser_offset_y} ${rear_laser_offset_z}" rpy="0 ${-PI} ${-1/4*PI}" />
+  		</xacro:sensor_sick_s300>
+  		<xacro:sensor_orbbec_astra prefix="$(arg prefix)front_rgbd_camera" parent="$(arg prefix)base_link" prefix_topic="front_rgbd_camera">
+  			<origin xyz="${front_rgbd_camera_offset_x} ${front_rgbd_camera_offset_y} ${front_rgbd_camera_offset_z}" rpy="0 0 0"/>
+  		</xacro:sensor_orbbec_astra>
+		<!--xacro:sensor_zed prefix="$(arg prefix)front_rgbd_camera" parent="$(arg prefix)base_link" prefix_topic="front_rgbd_camera">
+  			<origin xyz="${front_rgbd_camera_offset_x} ${front_rgbd_camera_offset_y} ${front_rgbd_camera_offset_z}" rpy="0 0 0"/>
+  		</xacro:sensor_zed-->
+    </xacro:macro>
+    <!-- Gazebo ros control pluggins -->
+    <xacro:ros_control/>
+    <xacro:if value="$(arg ros_planar_move_plugin)">
+        <xacro:omni_steering prefix="$(arg prefix)" publish_tf="false"/>
+    </xacro:if>
+    <xacro:rbkairos prefix="$(arg prefix)" publish_bf="true" hq="true" load_kinematics_file="$(arg load_kinematics_file)"/>
 </robot>
