Commit message: Revert "description: update xacros to work with local config files"
This reverts commit aa516fce50da9ce9f7491c69755b04ad985b423c.

File: rbkairos_description/robots/rbkairos_ur10.urdf.xacro (robot description, xacro)
@@ -8,16 +8,5 @@
   	<xacro:include filename="$(find summit_xl_description)/urdf/bases/summit_xls_base.urdf.xacro" />
     <!-- Include UR-10 ARM -->
- <!--ur10e parameters files -->
-	  <xacro:arg name="joint_limit_params" default="$(find rbkairos_control)/config/ur/ur10e/joint_limits.yaml"/>
-	  <xacro:arg name="kinematics_params" default="$(find rbkairos_control)/config/ur/ur10e/default_kinematics.yaml"/>
-	  <xacro:arg name="physical_params" default="$(find rbkairos_control)/config/ur/ur10e/physical_parameters.yaml"/>
-	  <xacro:arg name="visual_params" default="$(find rbkairos_control)/config/ur/ur10e/visual_parameters.yaml"/>
-	  <!--common parameters -->
-	  <xacro:arg name="transmission_hw_interface" default="hardware_interface/PositionJointInterface" />
-	  <xacro:arg name="safety_limits" default="false" doc="If True, enable the safety limits controller"/>
-	  <xacro:arg name="safety_pos_margin" default="0.15" doc="The lower/upper limits in the safety controller" />
-	  <xacro:arg name="safety_k_position" default="20" doc="Used to set k position in the safety controller" />
-	<!-- import main macro -->
- 	<xacro:include filename="$(find ur_description)/urdf/ur_macro.xacro"/>
+	<xacro:include filename="$(find ur_description)/urdf/ur10.urdf.xacro" />
   	<!-- Import summit XL wheels -->
   	<xacro:include filename="$(find summit_xl_description)/urdf/wheels/omni_wheel.urdf.xacro" />
@@ -83,19 +72,27 @@
   		</xacro:omni_wheel>
         <!-- UR-10 ARM -->
-		<joint name="$(arg prefix)arm_base_joint" type="fixed">
-						<origin xyz="${arm_position_x} ${arm_position_y} ${arm_position_z}" rpy="${arm_orientation_r} ${arm_orientation_p} ${arm_orientation_y}"/>
-						<parent link="$(arg prefix)base_link" />
-						<child link="$(arg prefix)arm_base_link" />
-					</joint>
-		<xacro:ur_robot
-			 prefix="$(arg prefix)arm_"
-			 joint_limits_parameters_file="$(arg joint_limit_params)"
-			 kinematics_parameters_file="$(arg kinematics_params)"
-			 physical_parameters_file="$(arg physical_params)"
-			 visual_parameters_file="$(arg visual_params)"
-			 transmission_hw_interface="$(arg transmission_hw_interface)"
-			 safety_limits="$(arg safety_limits)"
-			 safety_pos_margin="$(arg safety_pos_margin)"
-			 safety_k_position="$(arg safety_k_position)"/>
+		<xacro:if value="$(arg load_kinematics_file)">
+            <xacro:ur10_robot prefix="$(arg prefix)arm_" joint_limited="true"
+            shoulder_pan_lower_limit="${-pi}" shoulder_pan_upper_limit="${pi}"
+            wrist_3_lower_limit="${-pi}" wrist_3_upper_limit="${pi}"
+            kinematics_file="${load_yaml('$(find rbkairos_control)/config/ur10_calibration.yaml')}">
+            </xacro:ur10_robot>
+            <joint name="$(arg prefix)arm_base_joint" type="fixed">
+                <origin xyz="${arm_position_x} ${arm_position_y} ${arm_position_z}" rpy="${arm_orientation_r} ${arm_orientation_p} ${arm_orientation_y}"/>
+                <parent link="$(arg prefix)base_link" />
+                <child link="$(arg prefix)arm_base_link" />
+            </joint>
+		</xacro:if>
+		<xacro:unless value="$(arg load_kinematics_file)">
+            <xacro:ur10_robot prefix="$(arg prefix)arm_" joint_limited="true"
+            shoulder_pan_lower_limit="${-pi}" shoulder_pan_upper_limit="${pi}"
+            wrist_3_lower_limit="${-pi}" wrist_3_upper_limit="${pi}">
+            </xacro:ur10_robot>
+            <joint name="$(arg prefix)arm_base_joint" type="fixed">
+            <origin xyz="${arm_position_x} ${arm_position_y} ${arm_position_z}" rpy="${arm_orientation_r} ${arm_orientation_p} ${arm_orientation_y}"/>
+            <parent link="$(arg prefix)base_link" />
+            <child link="$(arg prefix)arm_base_link" />
+            </joint>
+		</xacro:unless>
         <!-- IMU -->
   		<xacro:sensor_imu_hector prefix="$(arg prefix)imu" parent="$(arg prefix)base_link">

File: rbkairos_description/robots/rbkairos_ur5.urdf.xacro (robot description, xacro)
@@ -8,17 +8,5 @@
 	<xacro:include filename="$(find rbkairos_description)/urdf/bases/rbkairos_base.urdf.xacro" />
 	<!-- Include UR-5 ARM -->
-	<!--xacro:include filename="$(find ur_description)/urdf/ur10.urdf.xacro" /-->
-	  <!--ur10e parameters files -->
-	  <xacro:arg name="joint_limit_params" default="$(find rbkairos_control)/config/ur/ur5e/joint_limits.yaml"/>
-	  <xacro:arg name="kinematics_params" default="$(find rbkairos_control)/config/ur/ur5e/default_kinematics.yaml"/>
-	  <xacro:arg name="physical_params" default="$(find rbkairos_control)/config/ur/ur5e/physical_parameters.yaml"/>
-	  <xacro:arg name="visual_params" default="$(find rbkairos_control)/config/ur/ur5e/visual_parameters.yaml"/>
-	  <!--common parameters -->
-	  <xacro:arg name="transmission_hw_interface" default="hardware_interface/PositionJointInterface" />
-	  <xacro:arg name="safety_limits" default="false" doc="If True, enable the safety limits controller"/>
-	  <xacro:arg name="safety_pos_margin" default="0.15" doc="The lower/upper limits in the safety controller" />
-	  <xacro:arg name="safety_k_position" default="20" doc="Used to set k position in the safety controller" />
-	<!-- import main macro -->
- 	<xacro:include filename="$(find ur_description)/urdf/ur_macro.xacro"/>
+	<xacro:include filename="$(find ur_description)/urdf/ur5.urdf.xacro" />
 	<!-- Flag to select the high or low quality model -->
 	<xacro:property name="hq" value="true" />
@@ -40,19 +28,27 @@
 		<xacro:rbkairos_base prefix="$(arg prefix)" publish_bf="true" hq="true"/>
 		<!-- UR-5 ARM -->
-		<joint name="$(arg prefix)arm_base_joint" type="fixed">
-						<origin xyz="${arm_position_x} ${arm_position_y} ${arm_position_z}" rpy="${arm_orientation_r} ${arm_orientation_p} ${arm_orientation_y}"/>
-						<parent link="$(arg prefix)base_link" />
-						<child link="$(arg prefix)arm_base_link" />
-					</joint>
-		<xacro:ur_robot
-			 prefix="$(arg prefix)arm_"
-			 joint_limits_parameters_file="$(arg joint_limit_params)"
-			 kinematics_parameters_file="$(arg kinematics_params)"
-			 physical_parameters_file="$(arg physical_params)"
-			 visual_parameters_file="$(arg visual_params)"
-			 transmission_hw_interface="$(arg transmission_hw_interface)"
-			 safety_limits="$(arg safety_limits)"
-			 safety_pos_margin="$(arg safety_pos_margin)"
-			 safety_k_position="$(arg safety_k_position)"/>
+		<xacro:if value="$(arg load_kinematics_file)">
+        <xacro:ur5_robot prefix="$(arg prefix)arm_" joint_limited="true"
+          shoulder_pan_lower_limit="${-pi}" shoulder_pan_upper_limit="${pi}"
+          wrist_3_lower_limit="${-pi}" wrist_3_upper_limit="${pi}"
+          kinematics_file="${load_yaml('$(find rbkairos_control)/config/ur5_calibration.yaml')}">
+        </xacro:ur5_robot>
+        <joint name="$(arg prefix)arm_base_joint" type="fixed">
+          <origin xyz="${arm_position_x} ${arm_position_y} ${arm_position_z}" rpy="${arm_orientation_r} ${arm_orientation_p} ${arm_orientation_y}"/>
+          <parent link="$(arg prefix)base_link" />
+          <child link="$(arg prefix)arm_base_link" />
+        </joint>
+		</xacro:if>
+		<xacro:unless value="$(arg load_kinematics_file)">
+        <xacro:ur5_robot prefix="$(arg prefix)arm_" joint_limited="true"
+          shoulder_pan_lower_limit="${-pi}" shoulder_pan_upper_limit="${pi}"
+          wrist_3_lower_limit="${-pi}" wrist_3_upper_limit="${pi}">
+        </xacro:ur5_robot>
+        <joint name="$(arg prefix)arm_base_joint" type="fixed">
+          <origin xyz="${arm_position_x} ${arm_position_y} ${arm_position_z}" rpy="${arm_orientation_r} ${arm_orientation_p} ${arm_orientation_y}"/>
+          <parent link="$(arg prefix)base_link" />
+          <child link="$(arg prefix)arm_base_link" />
+        </joint>
+		</xacro:unless>
 	</xacro:macro>
    <!-- Gazebo ros control pluggins -->

File: rbkairos_description/robots/rbkairos_ur5_oem.urdf.xacro (robot description, xacro)
@@ -8,16 +8,5 @@
   	<xacro:include filename="$(find summit_xl_description)/urdf/bases/summit_xlsk_base_oem.urdf.xacro" />
     <!-- Include UR-5 ARM -->
-	  <!--ur10e parameters files -->
-	  <xacro:arg name="joint_limit_params" default="$(find rbkairos_control)/config/ur/ur5e/joint_limits.yaml"/>
-	  <xacro:arg name="kinematics_params" default="$(find rbkairos_control)/config/ur/ur5e/default_kinematics.yaml"/>
-	  <xacro:arg name="physical_params" default="$(find rbkairos_control)/config/ur/ur5e/physical_parameters.yaml"/>
-	  <xacro:arg name="visual_params" default="$(find rbkairos_control)/config/ur/ur5e/visual_parameters.yaml"/>
-	  <!--common parameters -->
-	  <xacro:arg name="transmission_hw_interface" default="hardware_interface/PositionJointInterface" />
-	  <xacro:arg name="safety_limits" default="false" doc="If True, enable the safety limits controller"/>
-	  <xacro:arg name="safety_pos_margin" default="0.15" doc="The lower/upper limits in the safety controller" />
-	  <xacro:arg name="safety_k_position" default="20" doc="Used to set k position in the safety controller" />
-	<!-- import main macro -->
- 	<xacro:include filename="$(find ur_description)/urdf/ur_macro.xacro"/>
+	<xacro:include filename="$(find ur_description)/urdf/ur5.urdf.xacro" />
   	<!-- Import summit XL wheels -->
   	<xacro:include filename="$(find summit_xl_description)/urdf/wheels/omni_wheel.urdf.xacro" />
@@ -83,19 +72,27 @@
   		</xacro:omni_wheel>
         <!-- UR-5 ARM -->
-		<joint name="$(arg prefix)arm_base_joint" type="fixed">
-						<origin xyz="${arm_position_x} ${arm_position_y} ${arm_position_z}" rpy="${arm_orientation_r} ${arm_orientation_p} ${arm_orientation_y}"/>
-						<parent link="$(arg prefix)base_link" />
-						<child link="$(arg prefix)arm_base_link" />
-					</joint>
-		<xacro:ur_robot
-			 prefix="$(arg prefix)arm_"
-			 joint_limits_parameters_file="$(arg joint_limit_params)"
-			 kinematics_parameters_file="$(arg kinematics_params)"
-			 physical_parameters_file="$(arg physical_params)"
-			 visual_parameters_file="$(arg visual_params)"
-			 transmission_hw_interface="$(arg transmission_hw_interface)"
-			 safety_limits="$(arg safety_limits)"
-			 safety_pos_margin="$(arg safety_pos_margin)"
-			 safety_k_position="$(arg safety_k_position)"/>
+		<xacro:if value="$(arg load_kinematics_file)">
+            <xacro:ur5_robot prefix="$(arg prefix)arm_" joint_limited="true"
+            shoulder_pan_lower_limit="${-pi}" shoulder_pan_upper_limit="${pi}"
+            wrist_3_lower_limit="${-pi}" wrist_3_upper_limit="${pi}"
+            kinematics_file="${load_yaml('$(find rbkairos_control)/config/ur5_calibration.yaml')}">
+            </xacro:ur5_robot>
+            <joint name="$(arg prefix)arm_base_joint" type="fixed">
+                <origin xyz="${arm_position_x} ${arm_position_y} ${arm_position_z}" rpy="${arm_orientation_r} ${arm_orientation_p} ${arm_orientation_y}"/>
+                <parent link="$(arg prefix)base_link" />
+                <child link="$(arg prefix)arm_base_link" />
+            </joint>
+		</xacro:if>
+		<xacro:unless value="$(arg load_kinematics_file)">
+            <xacro:ur5_robot prefix="$(arg prefix)arm_" joint_limited="true"
+            shoulder_pan_lower_limit="${-pi}" shoulder_pan_upper_limit="${pi}"
+            wrist_3_lower_limit="${-pi}" wrist_3_upper_limit="${pi}">
+            </xacro:ur5_robot>
+            <joint name="$(arg prefix)arm_base_joint" type="fixed">
+            <origin xyz="${arm_position_x} ${arm_position_y} ${arm_position_z}" rpy="${arm_orientation_r} ${arm_orientation_p} ${arm_orientation_y}"/>
+            <parent link="$(arg prefix)base_link" />
+            <child link="$(arg prefix)arm_base_link" />
+            </joint>
+		</xacro:unless>
         <!-- IMU -->
   		<xacro:sensor_imu_hector prefix="$(arg prefix)imu" parent="$(arg prefix)base_link">
