Commit message: description: Updates robots to work with latest UR repo version

File: rbkairos_description/robots/rbkairos_ur10e_plus.urdf.xacro (robot description, xacro)
@@ -6,5 +6,5 @@
   	<!-- First we import all posible elements defined in the urdf.xacro files. All these elements are defined as macro:xacros -->
   	<!-- Import summit XL base elements -->
-  	<xacro:include filename="$(find summit_xl_description)/urdf/bases/summit_xls_base.urdf.xacro" />
+  	<xacro:include filename="$(find summit_xl_description)/urdf/bases/summit_xlsk_base_plus.urdf.xacro" />
     <!-- Include UR-10 ARM -->
 	<xacro:include filename="$(find ur_description)/urdf/inc/ur10e_macro.xacro" />
@@ -48,5 +48,5 @@
     <xacro:property name="arm_position_x" value="0.0"/>
     <xacro:property name="arm_position_y" value="0"/>
-    <xacro:property name="arm_position_z" value="0.383612"/>
+    <xacro:property name="arm_position_z" value="0.56162"/>
     <xacro:property name="arm_orientation_r" value="0"/>
     <xacro:property name="arm_orientation_p" value="0"/>
@@ -71,12 +71,12 @@
   			<origin xyz="-${wheel_offset_x} -${wheel_offset_y} ${wheel_offset_z}" rpy="0 0 0"/>
   		</xacro:omni_wheel>
-        <!-- UR-10 ARM -->
-        <xacro:ur10e_robot prefix="$(arg prefix)arm_">
-        </xacro:ur10e_robot>
-        <joint name="$(arg prefix)arm_base_joint" type="fixed">
-            <origin xyz="${arm_position_x} ${arm_position_y} ${arm_position_z}" rpy="${arm_orientation_r} ${arm_orientation_p} ${arm_orientation_y}"/>
-            <parent link="$(arg prefix)base_link" />
-            <child link="$(arg prefix)arm_base_link" />
-        </joint>
+        <!-- UR-10e ARM -->
+            <xacro:ur10e_robot prefix="$(arg prefix)arm_">
+            </xacro:ur10e_robot>
+            <joint name="$(arg prefix)arm_base_joint" type="fixed">
+                <origin xyz="${arm_position_x} ${arm_position_y} ${arm_position_z}" rpy="${arm_orientation_r} ${arm_orientation_p} ${arm_orientation_y}"/>
+                <parent link="$(arg prefix)base_link" />
+                <child link="$(arg prefix)arm_base_link" />
+            </joint>
         <!-- IMU -->
   		<xacro:sensor_imu_hector prefix="$(arg prefix)imu" parent="$(arg prefix)base_link">

File: rbkairos_description/robots/rbkairos_ur5.urdf.xacro (robot description, xacro)
@@ -8,5 +8,5 @@
 	<xacro:include filename="$(find rbkairos_description)/urdf/bases/rbkairos_base.urdf.xacro" />
 	<!-- Include UR-5 ARM -->
-	<xacro:include filename="$(find ur_description)/urdf/ur5.urdf.xacro" />
+	<xacro:include filename="$(find ur_description)/urdf/inc/ur5_macro.xacro" />
 	<!-- Flag to select the high or low quality model -->
 	<xacro:property name="hq" value="true" />
@@ -28,27 +28,11 @@
 		<xacro:rbkairos_base prefix="$(arg prefix)" publish_bf="true" hq="true"/>
 		<!-- UR-5 ARM -->
-		<xacro:if value="$(arg load_kinematics_file)">
-        <xacro:ur5_robot prefix="$(arg prefix)arm_" joint_limited="true"
-          shoulder_pan_lower_limit="${-pi}" shoulder_pan_upper_limit="${pi}"
-          wrist_3_lower_limit="${-pi}" wrist_3_upper_limit="${pi}"
-          kinematics_file="${load_yaml('$(find rbkairos_control)/config/ur5_calibration.yaml')}">
-        </xacro:ur5_robot>
-        <joint name="$(arg prefix)arm_base_joint" type="fixed">
-          <origin xyz="${arm_position_x} ${arm_position_y} ${arm_position_z}" rpy="${arm_orientation_r} ${arm_orientation_p} ${arm_orientation_y}"/>
-          <parent link="$(arg prefix)base_link" />
-          <child link="$(arg prefix)arm_base_link" />
-        </joint>
-		</xacro:if>
-		<xacro:unless value="$(arg load_kinematics_file)">
-        <xacro:ur5_robot prefix="$(arg prefix)arm_" joint_limited="true"
-          shoulder_pan_lower_limit="${-pi}" shoulder_pan_upper_limit="${pi}"
-          wrist_3_lower_limit="${-pi}" wrist_3_upper_limit="${pi}">
-        </xacro:ur5_robot>
-        <joint name="$(arg prefix)arm_base_joint" type="fixed">
-          <origin xyz="${arm_position_x} ${arm_position_y} ${arm_position_z}" rpy="${arm_orientation_r} ${arm_orientation_p} ${arm_orientation_y}"/>
-          <parent link="$(arg prefix)base_link" />
-          <child link="$(arg prefix)arm_base_link" />
-        </joint>
-		</xacro:unless>
+    <xacro:ur5_robot prefix="$(arg prefix)arm_" >
+    </xacro:ur5_robot>
+    <joint name="$(arg prefix)arm_base_joint" type="fixed">
+      <origin xyz="${arm_position_x} ${arm_position_y} ${arm_position_z}" rpy="${arm_orientation_r} ${arm_orientation_p} ${arm_orientation_y}"/>
+      <parent link="$(arg prefix)base_link" />
+      <child link="$(arg prefix)arm_base_link" />
+    </joint>
 	</xacro:macro>
    <!-- Gazebo ros control pluggins -->

File: rbkairos_description/robots/rbkairos_ur5e_plus.urdf.xacro (robot description, xacro)
@@ -8,5 +8,5 @@
   	<xacro:include filename="$(find summit_xl_description)/urdf/bases/summit_xlsk_base_plus.urdf.xacro" />
     <!-- Include UR-5 ARM -->
-	<xacro:include filename="$(find ur_description)/urdf/ur5.urdf.xacro" />
+	<xacro:include filename="$(find ur_description)/urdf/inc/ur5e_macro.xacro" />
 	<!-- Include EGH Gripper-->
 	<xacro:include filename="$(find egh_gripper_description)/urdf/egh_gripper.urdf.xacro" />
@@ -74,27 +74,11 @@
   		</xacro:omni_wheel>
         <!-- UR-5 ARM -->
-		<xacro:if value="$(arg load_kinematics_file)">
-            <xacro:ur5_robot prefix="$(arg prefix)arm_" joint_limited="true"
-            shoulder_pan_lower_limit="${-pi}" shoulder_pan_upper_limit="${pi}"
-            wrist_3_lower_limit="${-pi}" wrist_3_upper_limit="${pi}"
-            kinematics_file="${load_yaml('$(find rbkairos_control)/config/ur5_calibration.yaml')}">
-            </xacro:ur5_robot>
-            <joint name="$(arg prefix)arm_base_joint" type="fixed">
-                <origin xyz="${arm_position_x} ${arm_position_y} ${arm_position_z}" rpy="${arm_orientation_r} ${arm_orientation_p} ${arm_orientation_y}"/>
-                <parent link="$(arg prefix)base_link" />
-                <child link="$(arg prefix)arm_base_link" />
-            </joint>
-		</xacro:if>
-		<xacro:unless value="$(arg load_kinematics_file)">
-            <xacro:ur5_robot prefix="$(arg prefix)arm_" joint_limited="true"
-            shoulder_pan_lower_limit="${-pi}" shoulder_pan_upper_limit="${pi}"
-            wrist_3_lower_limit="${-pi}" wrist_3_upper_limit="${pi}">
-            </xacro:ur5_robot>
-            <joint name="$(arg prefix)arm_base_joint" type="fixed">
-            <origin xyz="${arm_position_x} ${arm_position_y} ${arm_position_z}" rpy="${arm_orientation_r} ${arm_orientation_p} ${arm_orientation_y}"/>
-            <parent link="$(arg prefix)base_link" />
-            <child link="$(arg prefix)arm_base_link" />
-            </joint>
-		</xacro:unless>
+		<xacro:ur5e_robot prefix="$(arg prefix)arm_">
+		</xacro:ur5e_robot>
+		<joint name="$(arg prefix)arm_base_joint" type="fixed">
+			<origin xyz="${arm_position_x} ${arm_position_y} ${arm_position_z}" rpy="${arm_orientation_r} ${arm_orientation_p} ${arm_orientation_y}"/>
+			<parent link="$(arg prefix)base_link" />
+			<child link="$(arg prefix)arm_base_link" />
+		</joint>
         <!-- IMU -->
   		<xacro:sensor_imu_hector prefix="$(arg prefix)imu" parent="$(arg prefix)base_link">

Commit message: description: Updates laser positions and adds laser_support

File: rbkairos_description/robots/rbkairos_ur10e_plus.urdf.xacro (robot description, xacro)
@@ -17,13 +17,13 @@
   	<xacro:property name="PI" value="3.1415926535897931"/>
   	<!-- Wheel parameters -->
-  	<xacro:property name="wheel_offset_x" value="0.2225" />    <!-- x,y,z in translation from base_link to the center of the wheel -->
-  	<xacro:property name="wheel_offset_y" value="0.2045" />
+  	<xacro:property name="wheel_offset_x" value="0.21528" />    <!-- x,y,z in translation from base_link to the center of the wheel -->
+  	<xacro:property name="wheel_offset_y" value="0.2690" />
   	<xacro:property name="wheel_offset_z" value="0.0" />
-  	<xacro:property name="front_laser_offset_x" value="0.2865"/>
-  	<xacro:property name="front_laser_offset_y" value="-0.20894"/>
-  	<xacro:property name="front_laser_offset_z" value="0.2973"/>
-  	<xacro:property name="rear_laser_offset_x" value="-0.2865"/>
-  	<xacro:property name="rear_laser_offset_y" value="0.20894"/>
-  	<xacro:property name="rear_laser_offset_z" value="0.2973"/>
+	<xacro:property name="front_laser_offset_x" value="0.42109"/>
+  	<xacro:property name="front_laser_offset_y" value="-0.32737"/>
+  	<xacro:property name="front_laser_offset_z" value="0.16037"/>
+  	<xacro:property name="rear_laser_offset_x" value="-0.42109"/>
+  	<xacro:property name="rear_laser_offset_y" value="0.32737"/>
+  	<xacro:property name="rear_laser_offset_z" value="0.16037"/>
   	<xacro:property name="front_ptz_camera_offset_x" value="0.308"/>
   	<xacro:property name="front_ptz_camera_offset_y" value="0.141"/>
@@ -58,5 +58,5 @@
   		<!-- Here we create the robot elements using the xacro:macros imported at the beggining of this file -->
   		<!-- Summit XL base -->
-  		<xacro:summit_xls_base prefix="$(arg prefix)" publish_bf="true" hq="${hq}" />
+  		<xacro:summit_xls_base prefix="$(arg prefix)" publish_bf="true" hq="${hq}" laser_support="true" />
   		<xacro:omni_wheel prefix="$(arg prefix)front_right" parent="$(arg prefix)base_link" reflect="false" hq="${hq}">
   			<origin xyz="${wheel_offset_x} -${wheel_offset_y} ${wheel_offset_z}" rpy="0 0 0"/>

File: rbkairos_description/robots/rbkairos_ur5e_plus.urdf.xacro (robot description, xacro)
@@ -60,5 +60,5 @@
   		<!-- Here we create the robot elements using the xacro:macros imported at the beggining of this file -->
   		<!-- Summit XL base -->
-  		<xacro:summit_xls_base prefix="$(arg prefix)" publish_bf="true" hq="${hq}" />
+  		<xacro:summit_xls_base prefix="$(arg prefix)" publish_bf="true" hq="${hq}" laser_support="true"/>
   		<xacro:omni_wheel prefix="$(arg prefix)front_right" parent="$(arg prefix)base_link" reflect="false" hq="${hq}">
   			<origin xyz="${wheel_offset_x} -${wheel_offset_y} ${wheel_offset_z}" rpy="0 0 0"/>
