Commit message: description:rbkairos16: set microscan3 as default laser

File: rbkairos_description/robots/rbkairos_extension_ur16.urdf.xacro (robot description, xacro)
@@ -44,5 +44,5 @@
   	<xacro:property name="rear_ptz_camera_offset_y" value="-0.141"/>
   	<xacro:property name="rear_ptz_camera_offset_z" value="0.195"/>
-	<xacro:property name="ur_support_offset_x" value="0.189"/>
+	  <xacro:property name="ur_support_offset_x" value="0.189"/>
   	<xacro:property name="ur_support_offset_y" value="0.0"/>
   	<xacro:property name="ur_support_offset_z" value="0.38212"/>
@@ -107,10 +107,10 @@
   		</xacro:sensor_imu_hector>
   		<!-- SENSORS -->
-  		<xacro:sensor_sick_s300 prefix="$(arg prefix)front_laser" parent="$(arg prefix)base_link" prefix_topic="front_laser">
+  		<xacro:sensor_sick_microscan3 prefix="$(arg prefix)front_laser" parent="$(arg prefix)base_link" prefix_topic="front_laser">
   			<origin xyz="${front_laser_offset_x} ${front_laser_offset_y} ${front_laser_offset_z}" rpy="0 ${-PI} ${3/4*PI}" />
-  		</xacro:sensor_sick_s300>
-  		<xacro:sensor_sick_s300 prefix="$(arg prefix)rear_laser" parent="$(arg prefix)base_link" prefix_topic="rear_laser">
+  		</xacro:sensor_sick_microscan3>
+  		<xacro:sensor_sick_microscan3 prefix="$(arg prefix)rear_laser" parent="$(arg prefix)base_link" prefix_topic="rear_laser">
   			<origin xyz="${rear_laser_offset_x} ${rear_laser_offset_y} ${rear_laser_offset_z}" rpy="0 ${-PI} ${-1/4*PI}" />
-  		</xacro:sensor_sick_s300>
+  		</xacro:sensor_sick_microscan3>
   		<xacro:sensor_orbbec_astra prefix="$(arg prefix)front_rgbd_camera" parent="$(arg prefix)base_link" prefix_topic="front_rgbd_camera">
   			<origin xyz="${front_rgbd_camera_offset_x} ${front_rgbd_camera_offset_y} ${front_rgbd_camera_offset_z}" rpy="0 0 0"/>

Commit message: description: update rbkairos16 default model

File: rbkairos_description/robots/rbkairos_extension_ur16.urdf.xacro (robot description, xacro)
@@ -34,8 +34,8 @@
   	<xacro:property name="front_laser_offset_x" value="0.2865"/>
   	<xacro:property name="front_laser_offset_y" value="-0.20894"/>
-  	<xacro:property name="front_laser_offset_z" value="0.2973"/>
+  	<xacro:property name="front_laser_offset_z" value="0.30547"/>
   	<xacro:property name="rear_laser_offset_x" value="-0.2865"/>
   	<xacro:property name="rear_laser_offset_y" value="0.20894"/>
-  	<xacro:property name="rear_laser_offset_z" value="0.2973"/>
+  	<xacro:property name="rear_laser_offset_z" value="0.30547"/>
   	<xacro:property name="front_ptz_camera_offset_x" value="0.308"/>
   	<xacro:property name="front_ptz_camera_offset_y" value="0.141"/>

Commit message: description: Updates UR includes and macros

File: rbkairos_description/robots/rbkairos_extension_ur16.urdf.xacro (robot description, xacro)
@@ -19,5 +19,5 @@
 	  <xacro:arg name="safety_k_position" default="20" doc="Used to set k position in the safety controller" />
 	<!-- import main macro -->
- 	<xacro:include filename="$(find ur_description)/urdf/ur_macro.xacro"/>
+	<xacro:include filename="$(find ur_description)/urdf/inc/ur16e_macro.xacro" />
 	<xacro:include filename="$(find rbkairos_description)/urdf/structures/extension_ur16e.urdf.xacro" />
   	<!-- Import summit XL wheels -->
@@ -86,20 +86,12 @@
   			<origin xyz="-${wheel_offset_x} -${wheel_offset_y} ${wheel_offset_z}" rpy="0 0 0"/>
   		</xacro:omni_wheel>
-				<!-- UR-16 ARM -->
-		<joint name="$(arg prefix)arm_base_joint" type="fixed">
-						<origin xyz="${arm_position_x} ${arm_position_y} ${arm_position_z}" rpy="${arm_orientation_r} ${arm_orientation_p} ${arm_orientation_y}"/>
-						<parent link="$(arg prefix)base_link" />
-						<child link="$(arg prefix)arm_base_link" />
-					</joint>
-		<xacro:ur_robot
-			 prefix="$(arg prefix)arm_"
-			 joint_limits_parameters_file="$(arg joint_limit_params)"
-			 kinematics_parameters_file="$(arg kinematics_params)"
-			 physical_parameters_file="$(arg physical_params)"
-			 visual_parameters_file="$(arg visual_params)"
-			 transmission_hw_interface="$(arg transmission_hw_interface)"
-			 safety_limits="$(arg safety_limits)"
-			 safety_pos_margin="$(arg safety_pos_margin)"
-			 safety_k_position="$(arg safety_k_position)"/>
+		<!-- UR-16 ARM -->
+		<xacro:ur16e_robot prefix="$(arg prefix)arm_" >
+    </xacro:ur16e_robot>
+    <joint name="$(arg prefix)arm_base_joint" type="fixed">
+      <origin xyz="${arm_position_x} ${arm_position_y} ${arm_position_z}" rpy="${arm_orientation_r} ${arm_orientation_p} ${arm_orientation_y}"/>
+      <parent link="$(arg prefix)base_link" />
+      <child link="$(arg prefix)arm_base_link" />
+    </joint>
         <!-- IMU -->
   		<xacro:sensor_imu_hector prefix="$(arg prefix)imu" parent="$(arg prefix)base_link">

File: rbkairos_description/robots/versions/rbkairos_ur10_vgc10.urdf.xacro (robot description, xacro)
@@ -8,5 +8,5 @@
   	<xacro:include filename="$(find summit_xl_description)/urdf/bases/summit_xls_base.urdf.xacro" />
     <!-- Include UR-10 ARM -->
-	  <xacro:include filename="$(find ur_description)/urdf/ur10.urdf.xacro" />
+	<xacro:include filename="$(find ur_description)/urdf/inc/ur10_macro.xacro" />
     <!-- Include OnRobot vgc10 -->
     <xacro:include filename="$(find rbkairos_description)/urdf/structures/vgc10.urdf.xacro" />
@@ -76,39 +76,11 @@
   		</xacro:omni_wheel>
       <!-- UR-10 ARM -->
-  		<!--xacro:if value="$(arg has_arm)">
-  			<xacro:ur10_robot prefix="$(arg prefix)arm_" joint_limited="true"
-  			shoulder_pan_lower_limit="${-pi}" shoulder_pan_upper_limit="${pi}"
-  			wrist_3_lower_limit="${-pi}" wrist_3_upper_limit="${pi}">
-  			</xacro:ur10_robot>
-  			<joint name="$(arg prefix)ur10_arm_base_joint" type="fixed">
-  				<origin xyz="0.0 0 0.4" rpy="0 0 ${PI*0}"/>
-  				<parent link="$(arg prefix)base_link" />
-  				<child link="$(arg prefix)arm_base_link" />
-  			</joint>
-  		</xacro:if-->
-      <!-- UR-10 ARM -->
-      <xacro:if value="$(arg load_kinematics_file)">
-          <xacro:ur10_robot prefix="$(arg prefix)arm_" joint_limited="true"
-          shoulder_pan_lower_limit="${-pi}" shoulder_pan_upper_limit="${pi}"
-          wrist_3_lower_limit="${-pi}" wrist_3_upper_limit="${pi}"
-          kinematics_file="${load_yaml('$(find rbkairos_control)/config/ur10_calibration.yaml')}">
-          </xacro:ur10_robot>
-          <joint name="$(arg prefix)arm_base_joint" type="fixed">
-              <origin xyz="${arm_position_x} ${arm_position_y} ${arm_position_z}" rpy="${arm_orientation_r} ${arm_orientation_p} ${arm_orientation_y}"/>
-              <parent link="$(arg prefix)base_link" />
-              <child link="$(arg prefix)arm_base_link" />
-          </joint>
-      </xacro:if>
-      <xacro:unless value="$(arg load_kinematics_file)">
-          <xacro:ur10_robot prefix="$(arg prefix)arm_" joint_limited="true"
-          shoulder_pan_lower_limit="${-pi}" shoulder_pan_upper_limit="${pi}"
-          wrist_3_lower_limit="${-pi}" wrist_3_upper_limit="${pi}">
-          </xacro:ur10_robot>
-          <joint name="$(arg prefix)arm_base_joint" type="fixed">
-          <origin xyz="${arm_position_x} ${arm_position_y} ${arm_position_z}" rpy="${arm_orientation_r} ${arm_orientation_p} ${arm_orientation_y}"/>
-          <parent link="$(arg prefix)base_link" />
-          <child link="$(arg prefix)arm_base_link" />
-          </joint>
-      </xacro:unless>
+      <xacro:ur10_robot prefix="$(arg prefix)arm_" >
+    </xacro:ur10_robot>
+    <joint name="$(arg prefix)arm_base_joint" type="fixed">
+      <origin xyz="${arm_position_x} ${arm_position_y} ${arm_position_z}" rpy="${arm_orientation_r} ${arm_orientation_p} ${arm_orientation_y}"/>
+      <parent link="$(arg prefix)base_link" />
+      <child link="$(arg prefix)arm_base_link" />
+    </joint>
       <!-- OnRobot VGC-10 -->
       <xacro:vgc10 prefix="$(arg prefix)vgc10" parent="$(arg prefix)arm_tool0">
@@ -139,4 +111,4 @@
         <xacro:vacuum_gripper/>
     </xacro:macro>
-    <!-- xacro:rbkairos_ur10_vgc10 prefix="$(arg prefix)" publish_bf="true" hq="true" load_kinematics_file="$(arg load_kinematics_file)"/-->
+    <xacro:rbkairos_ur10_vgc10 prefix="$(arg prefix)" publish_bf="true" hq="true" load_kinematics_file="$(arg load_kinematics_file)"/>
 </robot>

File: rbkairos_description/robots/versions/rbkairos_ur10_wsg50.urdf.xacro (robot description, xacro)
@@ -8,5 +8,5 @@
 	<xacro:include filename="$(find rbkairos_description)/urdf/bases/rbkairos_base.urdf.xacro" />
 	<!-- Include UR-10 ARM -->
-	<xacro:include filename="$(find ur_description)/urdf/ur10.urdf.xacro" />
+	<xacro:include filename="$(find ur_description)/urdf/inc/ur10_macro.xacro" />
     <!-- Import Schunk WSG-50 -->
 	<xacro:include filename="$(find wsg_50_simulation)/urdf/wsg_50.urdf.xacro"/>
@@ -31,27 +31,11 @@
 		<xacro:rbkairos_base prefix="$(arg prefix)" publish_bf="true" hq="true"/>
         <!-- UR-10 ARM -->
-		<xacro:if value="$(arg load_kinematics_file)">
-			<xacro:ur10_robot prefix="$(arg prefix)arm_" joint_limited="true"
-			shoulder_pan_lower_limit="${-pi}" shoulder_pan_upper_limit="${pi}"
-			wrist_3_lower_limit="${-pi}" wrist_3_upper_limit="${pi}"
-			kinematics_file="${load_yaml('$(find rbkairos_control)/config/ur10_calibration.yaml')}">
-			</xacro:ur10_robot>
-			<joint name="$(arg prefix)arm_base_joint" type="fixed">
-				<origin xyz="${arm_position_x} ${arm_position_y} ${arm_position_z}" rpy="${arm_orientation_r} ${arm_orientation_p} ${arm_orientation_y}"/>
-				<parent link="$(arg prefix)base_link" />
-				<child link="$(arg prefix)arm_base_link" />
-			</joint>
-		</xacro:if>
-		<xacro:unless value="$(arg load_kinematics_file)">
-			<xacro:ur10_robot prefix="$(arg prefix)arm_" joint_limited="true"
-			shoulder_pan_lower_limit="${-pi}" shoulder_pan_upper_limit="${pi}"
-			wrist_3_lower_limit="${-pi}" wrist_3_upper_limit="${pi}">
-			</xacro:ur10_robot>
-			<joint name="$(arg prefix)arm_base_joint" type="fixed">
-			<origin xyz="${arm_position_x} ${arm_position_y} ${arm_position_z}" rpy="${arm_orientation_r} ${arm_orientation_p} ${arm_orientation_y}"/>
-			<parent link="$(arg prefix)base_link" />
-			<child link="$(arg prefix)arm_base_link" />
-			</joint>
-		</xacro:unless>
+		<xacro:ur10_robot prefix="$(arg prefix)arm_" >
+    </xacro:ur10_robot>
+    <joint name="$(arg prefix)arm_base_joint" type="fixed">
+      <origin xyz="${arm_position_x} ${arm_position_y} ${arm_position_z}" rpy="${arm_orientation_r} ${arm_orientation_p} ${arm_orientation_y}"/>
+      <parent link="$(arg prefix)base_link" />
+      <child link="$(arg prefix)arm_base_link" />
+    </joint>
 		<!-- Schunk WSG-50 -->
 		<xacro:wsg_50_xacro name="$(arg prefix)wsg50" parent="$(arg prefix)arm_tool0" finger_length="0.023" finger_tip="0">
@@ -64,4 +48,4 @@
         </xacro:if>
 	</xacro:macro>
-   <!-- xacro:rbkairos_ur10_wsg50 prefix="$(arg prefix)" publish_bf="true" hq="true" load_kinematics_file="$(arg load_kinematics_file)"/-->
+   <xacro:rbkairos_ur10_wsg50 prefix="$(arg prefix)" publish_bf="true" hq="true" load_kinematics_file="$(arg load_kinematics_file)"/>
 </robot>

File: rbkairos_description/robots/versions/rbkairos_ur5_plus.urdf.xacro (robot description, xacro)
@@ -8,5 +8,5 @@
   	<xacro:include filename="$(find summit_xl_description)/urdf/bases/summit_xlsk_base_plus.urdf.xacro" />
     <!-- Include UR-5 ARM -->
-	<xacro:include filename="$(find ur_description)/urdf/ur5.urdf.xacro" />
+	<xacro:include filename="$(find ur_description)/urdf/inc/ur5_macro.xacro" />
 	<!-- Include OnRobot vgc10 -->
     <!--xacro:include filename="$(find rbkairos_description)/urdf/structures/vgc10.urdf.xacro" />
@@ -86,5 +86,5 @@
   		<!-- Here we create the robot elements using the xacro:macros imported at the beggining of this file -->
   		<!-- Summit XL base -->
-  		<xacro:summit_xls_base prefix="${prefix}" publish_bf="true" hq="${hq}" />
+  		<xacro:summit_xls_base prefix="${prefix}" publish_bf="true" hq="${hq}" laser_support="false"/>
   		<xacro:omni_wheel prefix="${prefix}front_right" parent="${prefix}base_link" reflect="false" hq="${hq}">
   			<origin xyz="${wheel_offset_x} -${wheel_offset_y} ${wheel_offset_z}" rpy="0 0 0"/>
@@ -100,27 +100,11 @@
   		</xacro:omni_wheel>
         <!-- UR-5 ARM -->
-		<xacro:if value="$(arg load_kinematics_file)">
-            <xacro:ur5_robot prefix="${prefix}arm_" joint_limited="true"
-            shoulder_pan_lower_limit="${-pi}" shoulder_pan_upper_limit="${pi}"
-            wrist_3_lower_limit="${-pi}" wrist_3_upper_limit="${pi}"
-            kinematics_file="${load_yaml('$(find rbkairos_control)/config/ur5_calibration.yaml')}">
-            </xacro:ur5_robot>
-            <joint name="${prefix}arm_base_joint" type="fixed">
-                <origin xyz="${arm_position_x} ${arm_position_y} ${arm_position_z}" rpy="${arm_orientation_r} ${arm_orientation_p} ${arm_orientation_y}"/>
-                <parent link="${prefix}base_link" />
-                <child link="${prefix}arm_base_link" />
-            </joint>
-		</xacro:if>
-		<xacro:unless value="$(arg load_kinematics_file)">
-            <xacro:ur5_robot prefix="${prefix}arm_" joint_limited="true"
-            shoulder_pan_lower_limit="${-pi}" shoulder_pan_upper_limit="${pi}"
-            wrist_3_lower_limit="${-pi}" wrist_3_upper_limit="${pi}">
-            </xacro:ur5_robot>
-            <joint name="${prefix}arm_base_joint" type="fixed">
-            <origin xyz="${arm_position_x} ${arm_position_y} ${arm_position_z}" rpy="${arm_orientation_r} ${arm_orientation_p} ${arm_orientation_y}"/>
-            <parent link="${prefix}base_link" />
-            <child link="${prefix}arm_base_link" />
-            </joint>
-		</xacro:unless>
+		<xacro:ur5_robot prefix="$(arg prefix)arm_" >
+		</xacro:ur5_robot>
+		<joint name="${prefix}arm_base_joint" type="fixed">
+			<origin xyz="${arm_position_x} ${arm_position_y} ${arm_position_z}" rpy="${arm_orientation_r} ${arm_orientation_p} ${arm_orientation_y}"/>
+			<parent link="${prefix}base_link" />
+			<child link="${prefix}arm_base_link" />
+		</joint>
         <!-- OnRobot VGC-10 -->
         <!--xacro:vgc10 prefix="${prefix}vgc10" parent="${prefix}arm_tool0">
@@ -145,5 +129,5 @@
   		</xacro:sensor_zed-->
 		<!-- HOLDERS -->
-  		<xacro:holder prefix="${prefix}center_" parent="${prefix}base_link">
+  		<!--xacro:holder prefix="${prefix}center_" parent="${prefix}base_link">
   			<origin xyz="${center_holder_offset_x} ${center_holder_offset_y} ${center_holder_offset_z}" rpy="0 0 0"/>
   		</xacro:holder>
@@ -153,5 +137,5 @@
   		<xacro:holder prefix="${prefix}right_" parent="${prefix}base_link">
   			<origin xyz="${right_holder_offset_x} ${right_holder_offset_y} ${right_holder_offset_z}" rpy="0 0 0"/>
-  		</xacro:holder>
+  		</xacro:holder-->
         <!-- Intel Realsense support-->
         <!--xacro:realsense2vgc10_support prefix="$(arg prefix)wrist_rgbd_support" parent="$(arg prefix)arm_tool0">

File: rbkairos_description/robots/versions/rbkairos_ur5_plus_vgc10.urdf.xacro (robot description, xacro)
@@ -8,5 +8,5 @@
   	<xacro:include filename="$(find summit_xl_description)/urdf/bases/summit_xlsk_base_plus.urdf.xacro" />
     <!-- Include UR-5 ARM -->
-	<xacro:include filename="$(find ur_description)/urdf/ur5.urdf.xacro" />
+	<xacro:include filename="$(find ur_description)/urdf/inc/ur5_macro.xacro" />
 	<!-- Include OnRobot vgc10 -->
     <xacro:include filename="$(find rbkairos_description)/urdf/structures/vgc10.urdf.xacro" />
@@ -86,5 +86,5 @@
   		<!-- Here we create the robot elements using the xacro:macros imported at the beggining of this file -->
   		<!-- Summit XL base -->
-  		<xacro:summit_xls_base prefix="${prefix}" publish_bf="true" hq="${hq}" />
+  		<xacro:summit_xls_base prefix="${prefix}" publish_bf="true" hq="${hq}" laser_support="false"/>
   		<xacro:omni_wheel prefix="${prefix}front_right" parent="${prefix}base_link" reflect="false" hq="${hq}">
   			<origin xyz="${wheel_offset_x} -${wheel_offset_y} ${wheel_offset_z}" rpy="0 0 0"/>
@@ -100,27 +100,11 @@
   		</xacro:omni_wheel>
         <!-- UR-5 ARM -->
-		<xacro:if value="$(arg load_kinematics_file)">
-            <xacro:ur5_robot prefix="${prefix}arm_" joint_limited="true"
-            shoulder_pan_lower_limit="${-pi}" shoulder_pan_upper_limit="${pi}"
-            wrist_3_lower_limit="${-pi}" wrist_3_upper_limit="${pi}"
-            kinematics_file="${load_yaml('$(find rbkairos_control)/config/ur5_calibration.yaml')}">
-            </xacro:ur5_robot>
-            <joint name="${prefix}arm_base_joint" type="fixed">
-                <origin xyz="${arm_position_x} ${arm_position_y} ${arm_position_z}" rpy="${arm_orientation_r} ${arm_orientation_p} ${arm_orientation_y}"/>
-                <parent link="${prefix}base_link" />
-                <child link="${prefix}arm_base_link" />
-            </joint>
-		</xacro:if>
-		<xacro:unless value="$(arg load_kinematics_file)">
-            <xacro:ur5_robot prefix="${prefix}arm_" joint_limited="true"
-            shoulder_pan_lower_limit="${-pi}" shoulder_pan_upper_limit="${pi}"
-            wrist_3_lower_limit="${-pi}" wrist_3_upper_limit="${pi}">
-            </xacro:ur5_robot>
-            <joint name="${prefix}arm_base_joint" type="fixed">
-            <origin xyz="${arm_position_x} ${arm_position_y} ${arm_position_z}" rpy="${arm_orientation_r} ${arm_orientation_p} ${arm_orientation_y}"/>
-            <parent link="${prefix}base_link" />
-            <child link="${prefix}arm_base_link" />
-            </joint>
-		</xacro:unless>
+		<xacro:ur5_robot prefix="$(arg prefix)arm_" >
+    	</xacro:ur5_robot>
+		<joint name="${prefix}arm_base_joint" type="fixed">
+			<origin xyz="${arm_position_x} ${arm_position_y} ${arm_position_z}" rpy="${arm_orientation_r} ${arm_orientation_p} ${arm_orientation_y}"/>
+			<parent link="${prefix}base_link" />
+			<child link="${prefix}arm_base_link" />
+		</joint>
         <!-- OnRobot VGC-10 -->
         <xacro:vgc10 prefix="${prefix}vgc10" parent="${prefix}arm_tool0">

File: rbkairos_description/robots/versions/rbkairos_ur5_wsg50.urdf.xacro (robot description, xacro)
@@ -8,5 +8,5 @@
 	<xacro:include filename="$(find rbkairos_description)/robots/versions/rbkairos_ur5_wsg50_base.urdf.xacro"/>
 	<!-- Include UR-5 ARM -->
-	<xacro:include filename="$(find ur_description)/urdf/ur5.urdf.xacro"/>
+	<xacro:include filename="$(find ur_description)/urdf/inc/ur5_macro.xacro" />
   <!-- Import Schunk WSG-50 -->
 	<xacro:include filename="$(find rbkairos_description)/urdf/structures/wsg_50_support.urdf.xacro"/>
@@ -33,27 +33,11 @@
 		<xacro:rbkairos_base prefix="$(arg prefix)" publish_bf="true" hq="true"/>
 		<!-- UR-5 ARM -->
-		<xacro:if value="$(arg load_kinematics_file)">
-        <xacro:ur5_robot prefix="$(arg prefix)arm_" joint_limited="true"
-          shoulder_pan_lower_limit="${-pi}" shoulder_pan_upper_limit="${pi}"
-          wrist_3_lower_limit="${-pi}" wrist_3_upper_limit="${pi}"
-          kinematics_file="${load_yaml('$(find rbkairos_control)/config/ur5_calibration.yaml')}">
-        </xacro:ur5_robot>
-        <joint name="$(arg prefix)arm_base_joint" type="fixed">
-          <origin xyz="${arm_position_x} ${arm_position_y} ${arm_position_z}" rpy="${arm_orientation_r} ${arm_orientation_p} ${arm_orientation_y}"/>
-          <parent link="$(arg prefix)base_link" />
-          <child link="$(arg prefix)arm_base_link" />
-        </joint>
-		</xacro:if>
-		<xacro:unless value="$(arg load_kinematics_file)">
-        <xacro:ur5_robot prefix="$(arg prefix)arm_" joint_limited="true"
-          shoulder_pan_lower_limit="${-pi}" shoulder_pan_upper_limit="${pi}"
-          wrist_3_lower_limit="${-pi}" wrist_3_upper_limit="${pi}">
-        </xacro:ur5_robot>
-        <joint name="$(arg prefix)arm_base_joint" type="fixed">
-          <origin xyz="${arm_position_x} ${arm_position_y} ${arm_position_z}" rpy="${arm_orientation_r} ${arm_orientation_p} ${arm_orientation_y}"/>
-          <parent link="$(arg prefix)base_link" />
-          <child link="$(arg prefix)arm_base_link" />
-        </joint>
-		</xacro:unless>
+		<xacro:ur5_robot prefix="$(arg prefix)arm_" >
+    </xacro:ur5_robot>
+    <joint name="$(arg prefix)arm_base_joint" type="fixed">
+      <origin xyz="${arm_position_x} ${arm_position_y} ${arm_position_z}" rpy="${arm_orientation_r} ${arm_orientation_p} ${arm_orientation_y}"/>
+      <parent link="$(arg prefix)base_link" />
+      <child link="$(arg prefix)arm_base_link" />
+    </joint>
     <!-- Schunk Support -->
     <xacro:wsg50_support prefix="$(arg prefix)wsg50_support" parent="$(arg prefix)wrist_rgbd_support_link">
@@ -78,4 +62,4 @@
   </xacro:if>
 	</xacro:macro>
-  <!-- xacro:rbkairos_ur5_wsg50 prefix="$(arg prefix)" publish_bf="true" hq="true" load_kinematics_file="$(arg load_kinematics_file)"/-->
+  <xacro:rbkairos_ur5_wsg50 prefix="$(arg prefix)" publish_bf="true" hq="true" load_kinematics_file="$(arg load_kinematics_file)"/>
 </robot>

File: rbkairos_description/robots/versions/rbkairos_ur5_wsg50_base.urdf.xacro (robot description, xacro)
@@ -74,7 +74,7 @@
   			<origin xyz="${rear_laser_offset_x} ${rear_laser_offset_y} ${rear_laser_offset_z}" rpy="0 ${-PI} ${-1/4*PI}" />
   		</xacro:sensor_sick_s300>
-  		<xacro:sensor_zed prefix="$(arg prefix)front_rgbd_camera" parent="$(arg prefix)base_link" prefix_topic="front_rgbd_camera">
+  		<!--xacro:sensor_zed prefix="$(arg prefix)front_rgbd_camera" parent="$(arg prefix)base_link" prefix_topic="front_rgbd_camera">
   			<origin xyz="${front_rgbd_camera_offset_x} ${front_rgbd_camera_offset_y} ${front_rgbd_camera_offset_z}" rpy="0 0 0"/>
-  		</xacro:sensor_zed>
+  		</xacro:sensor_zed-->
      </xacro:macro>
 </robot>
