Commit message: description: adds gpu argument for sim

File: rbkairos_description/robots/rbkairos_base.urdf.xacro (robot description, xacro)
@@ -7,7 +7,8 @@
   <xacro:arg name="prefix" default="robot"/>
   <xacro:arg name="ros_planar_move_plugin" default="true"/>
+  <xacro:arg name="use_gpu_for_simulation" default="false"/>
   <!-- Import summit XL base elements -->
   <xacro:include filename="$(find rbkairos_description)/urdf/bases/rbkairos_base.urdf.xacro" />
-  <xacro:rbkairos_base prefix="$(arg prefix)" publish_bf="true" hq="true"/>
+  <xacro:rbkairos_base prefix="$(arg prefix)" publish_bf="true" hq="true" gpu="$(arg use_gpu_for_simulation)"/>
   <xacro:ros_control/>
   <xacro:if value="$(arg ros_planar_move_plugin)">

File: rbkairos_description/robots/rbkairos_extension_ur16.urdf.xacro (robot description, xacro)
@@ -61,4 +61,5 @@
   <xacro:arg name="ros_planar_move_plugin" default="false"/>
   <xacro:arg name="load_kinematics_file" default="false"/> <!-- Necesarry for ur_description compatible with official ur drivers-->
+  <xacro:arg name="use_gpu_for_simulation" default="false"/>
   <xacro:property name="arm_position_x" value="0.189"/>
   <xacro:property name="arm_position_y" value="0"/>
@@ -67,5 +68,5 @@
   <xacro:property name="arm_orientation_p" value="0"/>
   <xacro:property name="arm_orientation_y" value="${pi}"/>
-  <xacro:macro name="rbkairos" params="prefix publish_bf hq load_kinematics_file">
+  <xacro:macro name="rbkairos" params="prefix publish_bf hq load_kinematics_file gpu:=false">
     <!-- *************** -->
     <!-- Robots Elements -->
@@ -99,8 +100,8 @@
     </xacro:sensor_imu_hector>
     <!-- SENSORS -->
-    <xacro:sensor_sick_microscan3 prefix="$(arg prefix)front_laser" parent="$(arg prefix)base_link" prefix_topic="front_laser">
+    <xacro:sensor_sick_microscan3 prefix="$(arg prefix)front_laser" parent="$(arg prefix)base_link" prefix_topic="front_laser" gpu="${gpu}">
       <origin xyz="${front_laser_offset_x} ${front_laser_offset_y} ${front_laser_offset_z}" rpy="0 ${-PI} ${3/4*PI}" />
     </xacro:sensor_sick_microscan3>
-    <xacro:sensor_sick_microscan3 prefix="$(arg prefix)rear_laser" parent="$(arg prefix)base_link" prefix_topic="rear_laser">
+    <xacro:sensor_sick_microscan3 prefix="$(arg prefix)rear_laser" parent="$(arg prefix)base_link" prefix_topic="rear_laser" gpu="${gpu}">
       <origin xyz="${rear_laser_offset_x} ${rear_laser_offset_y} ${rear_laser_offset_z}" rpy="0 ${-PI} ${-1/4*PI}" />
     </xacro:sensor_sick_microscan3>
@@ -120,4 +121,4 @@
       <xacro:omni_steering prefix="$(arg prefix)" publish_tf="true"/>
   </xacro:if>
-  <xacro:rbkairos prefix="$(arg prefix)" publish_bf="true" hq="true" load_kinematics_file="$(arg load_kinematics_file)"/>
+  <xacro:rbkairos prefix="$(arg prefix)" publish_bf="true" hq="true" load_kinematics_file="$(arg load_kinematics_file)" gpu="$(arg use_gpu_for_simulation)"/>
 </robot>

File: rbkairos_description/robots/rbkairos_iiwa_plus.urdf.xacro (robot description, xacro)
@@ -46,4 +46,5 @@
   <xacro:arg name="ros_planar_move_plugin" default="false"/>
   <xacro:arg name="load_kinematics_file" default="false"/> <!-- Necesarry for ur_description compatible with official ur drivers-->
+  <xacro:arg name="use_gpu_for_simulation" default="false"/>
   <xacro:property name="arm_position_x" value="0.19217"/>
   <xacro:property name="arm_position_y" value="0"/>
@@ -52,5 +53,5 @@
   <xacro:property name="arm_orientation_p" value="0"/>
   <xacro:property name="arm_orientation_y" value="0"/>
-  <xacro:macro name="rbkairos" params="prefix publish_bf hq load_kinematics_file">
+  <xacro:macro name="rbkairos" params="prefix publish_bf hq load_kinematics_file gpu:=false">
     <!-- *************** -->
     <!-- Robots Elements -->
@@ -80,8 +81,8 @@
     </xacro:sensor_imu_hector>
     <!-- SENSORS -->
-    <xacro:sensor_hokuyo_ust10lx prefix="$(arg prefix)front_laser" parent="$(arg prefix)base_link" prefix_topic="front_laser">
+    <xacro:sensor_hokuyo_ust10lx prefix="$(arg prefix)front_laser" parent="$(arg prefix)base_link" prefix_topic="front_laser" gpu="${gpu}">
       <origin xyz="${front_laser_offset_x} ${front_laser_offset_y} ${front_laser_offset_z}" rpy="0 ${-PI} ${3/4*PI}" />
     </xacro:sensor_hokuyo_ust10lx>
-    <xacro:sensor_hokuyo_ust10lx prefix="$(arg prefix)rear_laser" parent="$(arg prefix)base_link" prefix_topic="rear_laser">
+    <xacro:sensor_hokuyo_ust10lx prefix="$(arg prefix)rear_laser" parent="$(arg prefix)base_link" prefix_topic="rear_laser" gpu="${gpu}">
       <origin xyz="${rear_laser_offset_x} ${rear_laser_offset_y} ${rear_laser_offset_z}" rpy="0 ${-PI} ${-1/4*PI}" />
     </xacro:sensor_hokuyo_ust10lx>
@@ -98,4 +99,4 @@
     <xacro:omni_steering prefix="$(arg prefix)" publish_tf="false"/>
   </xacro:if>
-  <xacro:rbkairos prefix="$(arg prefix)" publish_bf="true" hq="true" load_kinematics_file="$(arg load_kinematics_file)"/>
+  <xacro:rbkairos prefix="$(arg prefix)" publish_bf="true" hq="true" load_kinematics_file="$(arg load_kinematics_file)" gpu="$(arg use_gpu_for_simulation)"/>
 </robot>

File: rbkairos_description/robots/rbkairos_ur10.urdf.xacro (robot description, xacro)
@@ -46,4 +46,5 @@
   <xacro:arg name="ros_planar_move_plugin" default="false"/>
   <xacro:arg name="load_kinematics_file" default="false"/> <!-- Necesarry for ur_description compatible with official ur drivers-->
+  <xacro:arg name="use_gpu_for_simulation" default="false"/>
   <xacro:property name="arm_position_x" value="0.0"/>
   <xacro:property name="arm_position_y" value="0"/>
@@ -52,5 +53,5 @@
   <xacro:property name="arm_orientation_p" value="0"/>
   <xacro:property name="arm_orientation_y" value="0"/>
-  <xacro:macro name="rbkairos" params="prefix publish_bf hq load_kinematics_file">
+  <xacro:macro name="rbkairos" params="prefix publish_bf hq load_kinematics_file gpu:=false">
     <!-- *************** -->
     <!-- Robots Elements -->
@@ -84,8 +85,8 @@
     </xacro:sensor_imu_hector>
     <!-- SENSORS -->
-    <xacro:sensor_sick_s300 prefix="$(arg prefix)front_laser" parent="$(arg prefix)base_link" prefix_topic="front_laser">
+    <xacro:sensor_sick_s300 prefix="$(arg prefix)front_laser" parent="$(arg prefix)base_link" prefix_topic="front_laser" gpu="${gpu}">
       <origin xyz="${front_laser_offset_x} ${front_laser_offset_y} ${front_laser_offset_z}" rpy="0 ${-PI} ${3/4*PI}" />
     </xacro:sensor_sick_s300>
-    <xacro:sensor_sick_s300 prefix="$(arg prefix)rear_laser" parent="$(arg prefix)base_link" prefix_topic="rear_laser">
+    <xacro:sensor_sick_s300 prefix="$(arg prefix)rear_laser" parent="$(arg prefix)base_link" prefix_topic="rear_laser" gpu="${gpu}">
       <origin xyz="${rear_laser_offset_x} ${rear_laser_offset_y} ${rear_laser_offset_z}" rpy="0 ${-PI} ${-1/4*PI}" />
     </xacro:sensor_sick_s300>
@@ -102,4 +103,4 @@
     <xacro:omni_steering prefix="$(arg prefix)" publish_tf="true"/>
   </xacro:if>
-  <xacro:rbkairos prefix="$(arg prefix)" publish_bf="true" hq="true" load_kinematics_file="$(arg load_kinematics_file)"/>
+  <xacro:rbkairos prefix="$(arg prefix)" publish_bf="true" hq="true" load_kinematics_file="$(arg load_kinematics_file)" gpu="$(arg use_gpu_for_simulation)"/>
 </robot>

File: rbkairos_description/robots/rbkairos_ur10e_plus.urdf.xacro (robot description, xacro)
@@ -46,4 +46,5 @@
   <xacro:arg name="ros_planar_move_plugin" default="false"/>
   <xacro:arg name="load_kinematics_file" default="false"/> <!-- Necesarry for ur_description compatible with official ur drivers-->
+  <xacro:arg name="use_gpu_for_simulation" default="false"/>
   <xacro:property name="arm_position_x" value="0.0"/>
   <xacro:property name="arm_position_y" value="0"/>
@@ -52,5 +53,5 @@
   <xacro:property name="arm_orientation_p" value="0"/>
   <xacro:property name="arm_orientation_y" value="0"/>
-  <xacro:macro name="rbkairos" params="prefix publish_bf hq load_kinematics_file">
+  <xacro:macro name="rbkairos" params="prefix publish_bf hq load_kinematics_file gpu:=false">
     <!-- *************** -->
     <!-- Robots Elements -->
@@ -84,8 +85,8 @@
     </xacro:sensor_imu_hector>
     <!-- SENSORS -->
-    <xacro:sensor_sick_s300 prefix="$(arg prefix)front_laser" parent="$(arg prefix)base_link" prefix_topic="front_laser">
+    <xacro:sensor_sick_s300 prefix="$(arg prefix)front_laser" parent="$(arg prefix)base_link" prefix_topic="front_laser" gpu="${gpu}">
       <origin xyz="${front_laser_offset_x} ${front_laser_offset_y} ${front_laser_offset_z}" rpy="0 ${-PI} ${3/4*PI}" />
     </xacro:sensor_sick_s300>
-    <xacro:sensor_sick_s300 prefix="$(arg prefix)rear_laser" parent="$(arg prefix)base_link" prefix_topic="rear_laser">
+    <xacro:sensor_sick_s300 prefix="$(arg prefix)rear_laser" parent="$(arg prefix)base_link" prefix_topic="rear_laser" gpu="${gpu}">
       <origin xyz="${rear_laser_offset_x} ${rear_laser_offset_y} ${rear_laser_offset_z}" rpy="0 ${-PI} ${-1/4*PI}" />
     </xacro:sensor_sick_s300>
@@ -102,4 +103,4 @@
     <xacro:omni_steering prefix="$(arg prefix)" publish_tf="true"/>
   </xacro:if>
-  <xacro:rbkairos prefix="$(arg prefix)" publish_bf="true" hq="true" load_kinematics_file="$(arg load_kinematics_file)"/>
+  <xacro:rbkairos prefix="$(arg prefix)" publish_bf="true" hq="true" load_kinematics_file="$(arg load_kinematics_file)" gpu="$(arg use_gpu_for_simulation)"/>
 </robot>

File: rbkairos_description/robots/rbkairos_ur5.urdf.xacro (robot description, xacro)
@@ -14,4 +14,5 @@
   <xacro:arg name="ros_planar_move_plugin" default="false"/>
   <xacro:arg name="load_kinematics_file" default="false"/> <!-- Necesarry for ur_description compatible with official ur drivers-->
+  <xacro:arg name="use_gpu_for_simulation" default="false"/>
   <xacro:property name="arm_position_x" value="0.1883"/>
   <xacro:property name="arm_position_y" value="0"/>
@@ -20,5 +21,5 @@
   <xacro:property name="arm_orientation_p" value="0"/>
   <xacro:property name="arm_orientation_y" value="0.0"/>
-  <xacro:macro name="rbkairos" params="prefix publish_bf hq load_kinematics_file">
+  <xacro:macro name="rbkairos" params="prefix publish_bf hq load_kinematics_file gpu:=false">
     <!-- *************** -->
     <!-- Robots Elements -->
@@ -26,5 +27,5 @@
     <!-- Here we create the robot elements using the xacro:macros imported at the beggining of this file -->
     <!-- RBKAIROS base -->
-    <xacro:rbkairos_base prefix="$(arg prefix)" publish_bf="true" hq="true"/>
+    <xacro:rbkairos_base prefix="$(arg prefix)" publish_bf="true" hq="true" gpu="${gpu}"/>
     <!-- UR-5 ARM -->
     <xacro:ur5_robot prefix="$(arg prefix)arm_" >
@@ -41,4 +42,4 @@
     <xacro:omni_steering prefix="$(arg prefix)" publish_tf="true"/>
   </xacro:if>
-  <xacro:rbkairos prefix="$(arg prefix)" publish_bf="true" hq="true" load_kinematics_file="$(arg load_kinematics_file)"/>
+  <xacro:rbkairos prefix="$(arg prefix)" publish_bf="true" hq="true" load_kinematics_file="$(arg load_kinematics_file)" gpu="$(arg use_gpu_for_simulation)"/>
 </robot>

File: rbkairos_description/robots/rbkairos_ur5e_plus.urdf.xacro (robot description, xacro)
@@ -48,4 +48,5 @@
   <xacro:arg name="ros_planar_move_plugin" default="false"/>
   <xacro:arg name="load_kinematics_file" default="false"/> <!-- Necesarry for ur_description compatible with official ur drivers-->
+  <xacro:arg name="use_gpu_for_simulation" default="false"/>
   <xacro:property name="arm_position_x" value="0.15887"/>
   <xacro:property name="arm_position_y" value="0"/>
@@ -54,5 +55,5 @@
   <xacro:property name="arm_orientation_p" value="0"/>
   <xacro:property name="arm_orientation_y" value="0"/>
-  <xacro:macro name="rbkairos" params="prefix publish_bf hq load_kinematics_file">
+  <xacro:macro name="rbkairos" params="prefix publish_bf hq load_kinematics_file gpu:=false">
     <!-- *************** -->
     <!-- Robots Elements -->
@@ -86,8 +87,8 @@
     </xacro:sensor_imu_hector>
     <!-- SENSORS -->
-    <xacro:sensor_sick_s300 prefix="$(arg prefix)front_laser" parent="$(arg prefix)base_link" prefix_topic="front_laser">
+    <xacro:sensor_sick_s300 prefix="$(arg prefix)front_laser" parent="$(arg prefix)base_link" prefix_topic="front_laser" gpu="${gpu}">
       <origin xyz="${front_laser_offset_x} ${front_laser_offset_y} ${front_laser_offset_z}" rpy="0 ${-PI} ${3/4*PI}" />
     </xacro:sensor_sick_s300>
-    <xacro:sensor_sick_s300 prefix="$(arg prefix)rear_laser" parent="$(arg prefix)base_link" prefix_topic="rear_laser">
+    <xacro:sensor_sick_s300 prefix="$(arg prefix)rear_laser" parent="$(arg prefix)base_link" prefix_topic="rear_laser" gpu="${gpu}">
       <origin xyz="${rear_laser_offset_x} ${rear_laser_offset_y} ${rear_laser_offset_z}" rpy="0 ${-PI} ${-1/4*PI}" />
     </xacro:sensor_sick_s300>
@@ -107,4 +108,4 @@
     <xacro:omni_steering prefix="$(arg prefix)" publish_tf="true"/>
   </xacro:if>
-  <xacro:rbkairos prefix="$(arg prefix)" publish_bf="true" hq="true" load_kinematics_file="$(arg load_kinematics_file)"/>
+  <xacro:rbkairos prefix="$(arg prefix)" publish_bf="true" hq="true" load_kinematics_file="$(arg load_kinematics_file)" gpu="$(arg use_gpu_for_simulation)"/>
 </robot>

File: rbkairos_description/robots/versions/rbkairos_ur10_vgc10.urdf.xacro (robot description, xacro)
@@ -50,4 +50,5 @@
   <xacro:arg name="load_kinematics_file" default="false"/> <!-- Necesarry for ur_description compatible with official ur drivers-->
   <xacro:arg name="has_arm" default="true"/>
+  <xacro:arg name="use_gpu_for_simulation" default="false"/>
   <xacro:property name="arm_position_x" value="0.0"/>
   <xacro:property name="arm_position_y" value="0"/>
@@ -56,5 +57,5 @@
   <xacro:property name="arm_orientation_p" value="0"/>
   <xacro:property name="arm_orientation_y" value="0"/>
-  <xacro:macro name="rbkairos_ur10_vgc10" params="prefix publish_bf hq load_kinematics_file">
+  <xacro:macro name="rbkairos_ur10_vgc10" params="prefix publish_bf hq load_kinematics_file gpu:=false">
     <!-- *************** -->
     <!-- Robots Elements -->
@@ -92,8 +93,8 @@
     </xacro:sensor_imu_hector>
     <!-- SENSORS -->
-    <xacro:sensor_sick_s300 prefix="$(arg prefix)front_laser" parent="$(arg prefix)base_link" prefix_topic="front_laser">
+    <xacro:sensor_sick_s300 prefix="$(arg prefix)front_laser" parent="$(arg prefix)base_link" prefix_topic="front_laser" gpu="${gpu}">
       <origin xyz="${front_laser_offset_x} ${front_laser_offset_y} ${front_laser_offset_z}" rpy="0 ${-PI} ${3/4*PI}" />
     </xacro:sensor_sick_s300>
-    <xacro:sensor_sick_s300 prefix="$(arg prefix)rear_laser" parent="$(arg prefix)base_link" prefix_topic="rear_laser">
+    <xacro:sensor_sick_s300 prefix="$(arg prefix)rear_laser" parent="$(arg prefix)base_link" prefix_topic="rear_laser" gpu="${gpu}">
       <origin xyz="${rear_laser_offset_x} ${rear_laser_offset_y} ${rear_laser_offset_z}" rpy="0 ${-PI} ${-1/4*PI}" />
     </xacro:sensor_sick_s300>
@@ -111,4 +112,4 @@
     <xacro:vacuum_gripper/>
   </xacro:macro>
-  <xacro:rbkairos_ur10_vgc10 prefix="$(arg prefix)" publish_bf="true" hq="true" load_kinematics_file="$(arg load_kinematics_file)"/>
+  <xacro:rbkairos_ur10_vgc10 prefix="$(arg prefix)" publish_bf="true" hq="true" load_kinematics_file="$(arg load_kinematics_file)" gpu="$(arg use_gpu_for_simulation)"/>
 </robot>

File: rbkairos_description/robots/versions/rbkairos_ur10_wsg50.urdf.xacro (robot description, xacro)
@@ -17,4 +17,5 @@
   <xacro:arg name="has_arm" default="true"/>
   <xacro:arg name="load_kinematics_file" default="false"/> <!-- Necesarry for ur_description compatible with official ur drivers-->
+  <xacro:arg name="use_gpu_for_simulation" default="false"/>
   <xacro:property name="arm_position_x" value="0.0"/>
   <xacro:property name="arm_position_y" value="0"/>
@@ -23,5 +24,5 @@
   <xacro:property name="arm_orientation_p" value="0"/>
   <xacro:property name="arm_orientation_y" value="0"/>
-  <xacro:macro name="rbkairos_ur10_wsg50" params="prefix publish_bf hq load_kinematics_file">
+  <xacro:macro name="rbkairos_ur10_wsg50" params="prefix publish_bf hq load_kinematics_file gpu:=false">
   <!-- *************** -->
   <!-- Robots Elements -->
@@ -29,5 +30,5 @@
   <!-- Here we create the robot elements using the xacro:macros imported at the beggining of this file -->
   <!-- RBKAIROS base -->
-  <xacro:rbkairos_base prefix="$(arg prefix)" publish_bf="true" hq="true"/>
+  <xacro:rbkairos_base prefix="$(arg prefix)" publish_bf="true" hq="true" gpu="${gpu}"/>
     <!-- UR-10 ARM -->
     <xacro:ur10_robot prefix="$(arg prefix)arm_" >
@@ -48,4 +49,4 @@
     </xacro:if>
   </xacro:macro>
-  <xacro:rbkairos_ur10_wsg50 prefix="$(arg prefix)" publish_bf="true" hq="true" load_kinematics_file="$(arg load_kinematics_file)"/>
+  <xacro:rbkairos_ur10_wsg50 prefix="$(arg prefix)" publish_bf="true" hq="true" load_kinematics_file="$(arg load_kinematics_file)" gpu="$(arg use_gpu_for_simulation)"/>
 </robot>

File: rbkairos_description/robots/versions/rbkairos_ur5_egh.urdf.xacro (robot description, xacro)
@@ -18,4 +18,5 @@
   <xacro:arg name="ros_planar_move_plugin" default="false"/>
   <xacro:arg name="load_kinematics_file" default="false"/> <!-- Necesarry for ur_description compatible with official ur drivers-->
+  <xacro:arg name="use_gpu_for_simulation" default="false"/>
   <xacro:property name="arm_position_x" value="0.1883"/>
   <xacro:property name="arm_position_y" value="0"/>
@@ -24,5 +25,5 @@
   <xacro:property name="arm_orientation_p" value="0"/>
   <xacro:property name="arm_orientation_y" value="${3*pi/4}"/>
-  <xacro:macro name="rbkairos_ur5_egh" params="prefix publish_bf hq load_kinematics_file">
+  <xacro:macro name="rbkairos_ur5_egh" params="prefix publish_bf hq load_kinematics_file gpu:=false">
     <!-- *************** -->
     <!-- Robots Elements -->
@@ -30,5 +31,5 @@
     <!-- Here we create the robot elements using the xacro:macros imported at the beggining of this file -->
     <!-- RBKAIROS base -->
-    <xacro:rbkairos_base prefix="$(arg prefix)" publish_bf="true" hq="true"/>
+    <xacro:rbkairos_base prefix="$(arg prefix)" publish_bf="true" hq="true" gpu="${gpu}"/>
     <!-- UR-5 ARM -->
     <xacro:ur5_robot prefix="$(arg prefix)arm_" >
@@ -53,4 +54,4 @@
     </xacro:if>
   </xacro:macro>
-  <xacro:rbkairos_ur5_egh prefix="$(arg prefix)" publish_bf="true" hq="true" load_kinematics_file="$(arg load_kinematics_file)"/>
+  <xacro:rbkairos_ur5_egh prefix="$(arg prefix)" publish_bf="true" hq="true" load_kinematics_file="$(arg load_kinematics_file)" gpu="$(arg use_gpu_for_simulation)"/>
 </robot>

File: rbkairos_description/robots/versions/rbkairos_ur5_plus.urdf.xacro (robot description, xacro)
@@ -74,4 +74,5 @@
   <xacro:arg name="ros_planar_move_plugin" default="false"/>
   <xacro:arg name="load_kinematics_file" default="false"/> <!-- Necesarry for ur_description compatible with official ur drivers-->
+  <xacro:arg name="use_gpu_for_simulation" default="false"/>
   <xacro:property name="arm_position_x" value="0.15887"/>
   <xacro:property name="arm_position_y" value="0"/>
@@ -80,5 +81,5 @@
   <xacro:property name="arm_orientation_p" value="0"/>
   <xacro:property name="arm_orientation_y" value="0"/>
-  <xacro:macro name="rbkairos" params="prefix publish_bf hq load_kinematics_file">
+  <xacro:macro name="rbkairos" params="prefix publish_bf hq load_kinematics_file gpu:=false">
     <!-- *************** -->
     <!-- Robots Elements -->
@@ -116,8 +117,8 @@
     </xacro:sensor_imu_hector>
     <!-- SENSORS -->
-    <xacro:sensor_sick_s300 prefix="${prefix}front_laser" parent="${prefix}base_link" prefix_topic="front_laser">
+    <xacro:sensor_sick_s300 prefix="${prefix}front_laser" parent="${prefix}base_link" prefix_topic="front_laser" gpu="${gpu}">
       <origin xyz="${front_laser_offset_x} ${front_laser_offset_y} ${front_laser_offset_z}" rpy="0 ${-PI} ${3/4*PI}" />
     </xacro:sensor_sick_s300>
-    <xacro:sensor_sick_s300 prefix="${prefix}rear_laser" parent="${prefix}base_link" prefix_topic="rear_laser">
+    <xacro:sensor_sick_s300 prefix="${prefix}rear_laser" parent="${prefix}base_link" prefix_topic="rear_laser" gpu="${gpu}">
       <origin xyz="${rear_laser_offset_x} ${rear_laser_offset_y} ${rear_laser_offset_z}" rpy="0 ${-PI} ${-1/4*PI}" />
     </xacro:sensor_sick_s300>
@@ -182,4 +183,4 @@
     <xacro:omni_steering prefix="$(arg prefix)" publish_tf="true"/>
   </xacro:if>
-  <xacro:rbkairos prefix="$(arg prefix)" publish_bf="true" hq="true" load_kinematics_file="$(arg load_kinematics_file)"/>
+  <xacro:rbkairos prefix="$(arg prefix)" publish_bf="true" hq="true" load_kinematics_file="$(arg load_kinematics_file)" gpu="$(arg use_gpu_for_simulation)"/>
 </robot>

File: rbkairos_description/robots/versions/rbkairos_ur5_plus_vgc10.urdf.xacro (robot description, xacro)
@@ -74,4 +74,5 @@
   <xacro:arg name="ros_planar_move_plugin" default="false"/>
   <xacro:arg name="load_kinematics_file" default="false"/> <!-- Necesarry for ur_description compatible with official ur drivers-->
+  <xacro:arg name="use_gpu_for_simulation" default="false"/>
   <xacro:property name="arm_position_x" value="0.15887"/>
   <xacro:property name="arm_position_y" value="0"/>
@@ -80,5 +81,5 @@
   <xacro:property name="arm_orientation_p" value="0"/>
   <xacro:property name="arm_orientation_y" value="0"/>
-  <xacro:macro name="rbkairos" params="prefix publish_bf hq load_kinematics_file">
+  <xacro:macro name="rbkairos" params="prefix publish_bf hq load_kinematics_file gpu:=false">
     <!-- *************** -->
     <!-- Robots Elements -->
@@ -116,8 +117,8 @@
     </xacro:sensor_imu_hector>
     <!-- SENSORS -->
-    <xacro:sensor_sick_s300 prefix="${prefix}front_laser" parent="${prefix}base_link" prefix_topic="front_laser">
+    <xacro:sensor_sick_s300 prefix="${prefix}front_laser" parent="${prefix}base_link" prefix_topic="front_laser" gpu="${gpu}">
       <origin xyz="${front_laser_offset_x} ${front_laser_offset_y} ${front_laser_offset_z}" rpy="0 ${-PI} ${3/4*PI}" />
     </xacro:sensor_sick_s300>
-    <xacro:sensor_sick_s300 prefix="${prefix}rear_laser" parent="${prefix}base_link" prefix_topic="rear_laser">
+    <xacro:sensor_sick_s300 prefix="${prefix}rear_laser" parent="${prefix}base_link" prefix_topic="rear_laser" gpu="${gpu}">
       <origin xyz="${rear_laser_offset_x} ${rear_laser_offset_y} ${rear_laser_offset_z}" rpy="0 ${-PI} ${-1/4*PI}" />
     </xacro:sensor_sick_s300>
@@ -182,4 +183,4 @@
     <xacro:omni_steering prefix="$(arg prefix)" publish_tf="true"/>
   </xacro:if>
-  <xacro:rbkairos prefix="$(arg prefix)" publish_bf="true" hq="true" load_kinematics_file="$(arg load_kinematics_file)"/>
+  <xacro:rbkairos prefix="$(arg prefix)" publish_bf="true" hq="true" load_kinematics_file="$(arg load_kinematics_file)" gpu="$(arg use_gpu_for_simulation)"/>
 </robot>
