Commit message: description: adds gpu argument for sim

File: rbkairos_description/robots/versions/rbkairos_ur5_wsg50.urdf.xacro (robot description, xacro)
@@ -19,4 +19,5 @@
   <xacro:arg name="ros_planar_move_plugin" default="false"/>
   <xacro:arg name="load_kinematics_file" default="false"/> <!-- Necesarry for ur_description compatible with official ur drivers-->
+  <xacro:arg name="use_gpu_for_simulation" default="false"/>
   <xacro:property name="arm_position_x" value="0.1883"/>
   <xacro:property name="arm_position_y" value="0"/>
@@ -25,5 +26,5 @@
   <xacro:property name="arm_orientation_p" value="0"/>
   <xacro:property name="arm_orientation_y" value="${pi}"/>
-  <xacro:macro name="rbkairos_ur5_wsg50" params="prefix publish_bf hq load_kinematics_file">
+  <xacro:macro name="rbkairos_ur5_wsg50" params="prefix publish_bf hq load_kinematics_file gpu:=false">
     <!-- *************** -->
     <!-- Robots Elements -->
@@ -31,5 +32,5 @@
     <!-- Here we create the robot elements using the xacro:macros imported at the beggining of this file -->
     <!-- RBKAIROS base -->
-    <xacro:rbkairos_base prefix="$(arg prefix)" publish_bf="true" hq="true"/>
+    <xacro:rbkairos_base prefix="$(arg prefix)" publish_bf="true" hq="true" gpu="${gpu}"/>
     <!-- UR-5 ARM -->
     <xacro:ur5_robot prefix="$(arg prefix)arm_" >
@@ -62,4 +63,4 @@
   </xacro:if>
   </xacro:macro>
-  <xacro:rbkairos_ur5_wsg50 prefix="$(arg prefix)" publish_bf="true" hq="true" load_kinematics_file="$(arg load_kinematics_file)"/>
+  <xacro:rbkairos_ur5_wsg50 prefix="$(arg prefix)" publish_bf="true" hq="true" load_kinematics_file="$(arg load_kinematics_file)" gpu="$(arg use_gpu_for_simulation)"/>
 </robot>

File: rbkairos_description/robots/versions/rbkairos_ur5_wsg50_base.urdf.xacro (robot description, xacro)
@@ -44,5 +44,6 @@
   <xacro:arg name="prefix" default="summit_xl_"/>
   <xacro:arg name="ros_planar_move_plugin" default="false"/>
-  <xacro:macro name="rbkairos_base" params="prefix publish_bf hq">
+  <xacro:arg name="use_gpu_for_simulation" default="false"/>
+  <xacro:macro name="rbkairos_base" params="prefix publish_bf hq gpu:=false">
     <!-- *************** -->
     <!-- Robots Elements -->
@@ -68,8 +69,8 @@
     </xacro:sensor_imu_hector>
     <!-- SENSORS -->
-    <xacro:sensor_sick_s300 prefix="$(arg prefix)front_laser" parent="$(arg prefix)base_link" prefix_topic="front_laser">
+    <xacro:sensor_sick_s300 prefix="$(arg prefix)front_laser" parent="$(arg prefix)base_link" prefix_topic="front_laser" gpu="${gpu}">
       <origin xyz="${front_laser_offset_x} ${front_laser_offset_y} ${front_laser_offset_z}" rpy="0 ${-PI} ${3/4*PI}" />
     </xacro:sensor_sick_s300>
-    <xacro:sensor_sick_s300 prefix="$(arg prefix)rear_laser" parent="$(arg prefix)base_link" prefix_topic="rear_laser">
+    <xacro:sensor_sick_s300 prefix="$(arg prefix)rear_laser" parent="$(arg prefix)base_link" prefix_topic="rear_laser" gpu="${gpu}">
       <origin xyz="${rear_laser_offset_x} ${rear_laser_offset_y} ${rear_laser_offset_z}" rpy="0 ${-PI} ${-1/4*PI}" />
     </xacro:sensor_sick_s300>

File: rbkairos_description/urdf/bases/rbkairos_base.urdf.xacro (robot description, xacro)
@@ -44,5 +44,5 @@
   	<xacro:arg name="prefix" default="summit_xl_"/>
   	<xacro:arg name="ros_planar_move_plugin" default="false"/>
-    <xacro:macro name="rbkairos_base" params="prefix publish_bf hq">
+    <xacro:macro name="rbkairos_base" params="prefix publish_bf hq gpu:=false">
   		<!-- *************** -->
   		<!-- Robots Elements -->
@@ -68,8 +68,8 @@
   		</xacro:sensor_imu_hector>
   		<!-- SENSORS -->
-  		<xacro:sensor_sick_s300 prefix="$(arg prefix)front_laser" parent="$(arg prefix)base_link" prefix_topic="front_laser">
+  		<xacro:sensor_sick_s300 prefix="$(arg prefix)front_laser" parent="$(arg prefix)base_link" prefix_topic="front_laser" gpu="${gpu}">
   			<origin xyz="${front_laser_offset_x} ${front_laser_offset_y} ${front_laser_offset_z}" rpy="0 ${-PI} ${3/4*PI}" />
   		</xacro:sensor_sick_s300>
-  		<xacro:sensor_sick_s300 prefix="$(arg prefix)rear_laser" parent="$(arg prefix)base_link" prefix_topic="rear_laser">
+  		<xacro:sensor_sick_s300 prefix="$(arg prefix)rear_laser" parent="$(arg prefix)base_link" prefix_topic="rear_laser" gpu="${gpu}">
   			<origin xyz="${rear_laser_offset_x} ${rear_laser_offset_y} ${rear_laser_offset_z}" rpy="0 ${-PI} ${-1/4*PI}" />
   		</xacro:sensor_sick_s300>
