Commit message: Fixes rbkairos_5_plus_config   - Updates urdf file references   - Increase arm z position to avoid autocollision in moveit

File: rbkairos_description/robots/rbkairos_ur5e_plus.urdf.xacro (robot description, xacro)
@@ -51,5 +51,5 @@
   <xacro:property name="arm_position_x" value="0.15887"/>
   <xacro:property name="arm_position_y" value="0"/>
-  <xacro:property name="arm_position_z" value="0.56162"/>
+  <xacro:property name="arm_position_z" value="0.56362"/>
   <xacro:property name="arm_orientation_r" value="0"/>
   <xacro:property name="arm_orientation_p" value="0"/>
