Commit message: rbkairos_description: now you have to instance the macro when adding a robot

File: rbkairos_description/robots/versions/rbkairos_ur10_vgc10.urdf.xacro (robot description, xacro)
@@ -56,5 +56,5 @@
     <xacro:property name="arm_orientation_p" value="0"/>
     <xacro:property name="arm_orientation_y" value="0"/>
-    <xacro:macro name="rbkairos" params="prefix publish_bf hq load_kinematics_file">
+    <xacro:macro name="rbkairos_ur10_vgc10" params="prefix publish_bf hq load_kinematics_file">
   		<!-- *************** -->
   		<!-- Robots Elements -->
@@ -132,11 +132,11 @@
   			<origin xyz="${front_rgbd_camera_offset_x} ${front_rgbd_camera_offset_y} ${front_rgbd_camera_offset_z}" rpy="0 0 0"/>
   		</xacro:sensor_zed-->
+        <!-- Gazebo ros control pluggins -->
+        <xacro:ros_control/>
+        <xacro:if value="$(arg ros_planar_move_plugin)">
+            <xacro:omni_steering prefix="$(arg prefix)" publish_tf="true"/>
+        </xacro:if>
+        <xacro:vacuum_gripper/>
     </xacro:macro>
-    <!-- Gazebo ros control pluggins -->
-    <xacro:ros_control/>
-    <xacro:if value="$(arg ros_planar_move_plugin)">
-        <xacro:omni_steering prefix="$(arg prefix)" publish_tf="true"/>
-    </xacro:if>
-    <xacro:vacuum_gripper/>
-    <xacro:rbkairos prefix="$(arg prefix)" publish_bf="true" hq="true" load_kinematics_file="$(arg load_kinematics_file)"/>
+    <!-- xacro:rbkairos_ur10_vgc10 prefix="$(arg prefix)" publish_bf="true" hq="true" load_kinematics_file="$(arg load_kinematics_file)"/-->
 </robot>

File: rbkairos_description/robots/versions/rbkairos_ur10_wsg50.urdf.xacro (robot description, xacro)
@@ -23,5 +23,5 @@
     <xacro:property name="arm_orientation_p" value="0"/>
     <xacro:property name="arm_orientation_y" value="0"/>
-  <xacro:macro name="rbkairos" params="prefix publish_bf hq load_kinematics_file">
+    <xacro:macro name="rbkairos_ur10_wsg50" params="prefix publish_bf hq load_kinematics_file">
 		<!-- *************** -->
 		<!-- Robots Elements -->
@@ -58,10 +58,10 @@
 			<origin xyz="0.0 0.0 0.0" rpy="0 0 0"/>
 		</xacro:wsg_50_xacro>
+        <!-- Gazebo ros control pluggins -->
+        <xacro:ros_control/>
+        <xacro:if value="$(arg ros_planar_move_plugin)">
+            <xacro:omni_steering prefix="$(arg prefix)" publish_tf="true"/>
+        </xacro:if>
 	</xacro:macro>
-   <!-- Gazebo ros control pluggins -->
-   <xacro:ros_control/>
-   <xacro:if value="$(arg ros_planar_move_plugin)">
-	   <xacro:omni_steering prefix="$(arg prefix)" publish_tf="true"/>
-   </xacro:if>
-   <xacro:rbkairos prefix="$(arg prefix)" publish_bf="true" hq="true" load_kinematics_file="$(arg load_kinematics_file)"/>
+   <!-- xacro:rbkairos_ur10_wsg50 prefix="$(arg prefix)" publish_bf="true" hq="true" load_kinematics_file="$(arg load_kinematics_file)"/-->
 </robot>

File: rbkairos_description/robots/versions/rbkairos_ur5_egh.urdf.xacro (robot description, xacro)
@@ -24,5 +24,5 @@
   <xacro:property name="arm_orientation_p" value="0"/>
   <xacro:property name="arm_orientation_y" value="${3*pi/4}"/>
-  <xacro:macro name="rbkairos" params="prefix publish_bf hq load_kinematics_file">
+  <xacro:macro name="rbkairos_ur5_egh" params="prefix publish_bf hq load_kinematics_file">
 		<!-- *************** -->
 		<!-- Robots Elements -->
@@ -63,5 +63,4 @@
       <origin xyz="-0.075 0.0 0.065" rpy="0 ${-pi/2} 0"/>
     </xacro:sensor_r430>
-	</xacro:macro>
    <!-- Gazebo ros control pluggins -->
    <xacro:ros_control/>
@@ -69,4 +68,5 @@
 	   <xacro:omni_steering prefix="$(arg prefix)" publish_tf="true"/>
    </xacro:if>
-   <xacro:rbkairos prefix="$(arg prefix)" publish_bf="true" hq="true" load_kinematics_file="$(arg load_kinematics_file)"/>
+	</xacro:macro>
+   <!--xacro:rbkairos_ur10_wsg50 prefix="$(arg prefix)" publish_bf="true" hq="true" load_kinematics_file="$(arg load_kinematics_file)"/-->
 </robot>

File: rbkairos_description/robots/versions/rbkairos_ur5_oem_vgc10.urdf.xacro (robot description, xacro)
@@ -68,5 +68,5 @@
     <xacro:property name="arm_orientation_p" value="0"/>
     <xacro:property name="arm_orientation_y" value="0"/>
-    <xacro:macro name="rbkairos" params="prefix publish_bf hq load_kinematics_file">
+    <xacro:macro name="rbkairos_ur5_oem_vgc10" params="prefix publish_bf hq load_kinematics_file">
         <!-- *************** -->
         <!-- Robots Elements -->
@@ -133,11 +133,11 @@
         </xacro:sensor_zed-->
         <!-- Intel Realsense support-->
-        <!--xacro:realsense2vgc10_support prefix="$(arg prefix)wrist_rgbd_support" parent="$(arg prefix)arm_tool0">
+        <xacro:realsense2vgc10_support prefix="$(arg prefix)wrist_rgbd_support" parent="$(arg prefix)arm_tool0">
             <origin xyz="0.0 0.0 0.0" rpy="0 0 0.0"/>
-        </xacro:realsense2vgc10_support-->
+        </xacro:realsense2vgc10_support>
         <!-- Intel Realsense -->
-        <!--<xacro:sensor_intel_d435 prefix="$(arg prefix)wrist_rgbd" parent="$(arg prefix)arm_tool0" prefix_topic="wrist_rgbd">-->
-              <!--<origin xyz="0.07 0.0 0.065" rpy="${pi} ${-pi/2} 0"/>-->
-        <!--</xacro:sensor_intel_d435>-->
+        <xacro:sensor_intel_d435 prefix="$(arg prefix)wrist_rgbd" parent="$(arg prefix)wrist_rgbd_support_second_link" prefix_topic="wrist_rgbd" use_nominal_extrinsics="true" >
+              <origin xyz="0.07 0.0 0.065" rpy="${pi} ${-pi/2} 0"/>
+        </xacro:sensor_intel_d435>
       <gazebo>
         <plugin name="ground_truth_controller" filename="librobotnik_gazebo_ground_truth_odom.so">
@@ -170,5 +170,4 @@
         </plugin>
       </gazebo>
-    </xacro:macro>
     <!-- Gazebo ros control pluggins -->
     <xacro:ros_control/>
@@ -176,4 +175,4 @@
         <xacro:omni_steering prefix="$(arg prefix)" publish_tf="true"/>
     </xacro:if>
-    <xacro:rbkairos prefix="$(arg prefix)" publish_bf="true" hq="true" load_kinematics_file="$(arg load_kinematics_file)"/>
+    </xacro:macro>
 </robot>

File: rbkairos_description/robots/versions/rbkairos_ur5_wsg50.urdf.xacro (robot description, xacro)
@@ -25,5 +25,5 @@
   <xacro:property name="arm_orientation_p" value="0"/>
   <xacro:property name="arm_orientation_y" value="${pi}"/>
-  <xacro:macro name="rbkairos" params="prefix publish_bf hq load_kinematics_file">
+  <xacro:macro name="rbkairos_ur5_wsg50" params="prefix publish_bf hq load_kinematics_file">
 		<!-- *************** -->
 		<!-- Robots Elements -->
@@ -72,5 +72,4 @@
       <origin xyz="0.0515 0.0 0.065" rpy="${pi} ${-pi/2} 0"/>
     </xacro:sensor_r430>
-	</xacro:macro>
   <!-- Gazebo ros control pluggins -->
   <xacro:ros_control/>
@@ -78,4 +77,5 @@
     <xacro:omni_steering prefix="$(arg prefix)" publish_tf="true"/>
   </xacro:if>
-  <xacro:rbkairos prefix="$(arg prefix)" publish_bf="true" hq="true" load_kinematics_file="$(arg load_kinematics_file)"/>
+	</xacro:macro>
+  <!-- xacro:rbkairos_ur5_wsg50 prefix="$(arg prefix)" publish_bf="true" hq="true" load_kinematics_file="$(arg load_kinematics_file)"/-->
 </robot>
