Commit message: rbkairos_ur5_oem_vgc10.urdf.xacro: added intel d435 and its support

File: rbkairos_description/robots/versions/rbkairos_ur5_oem_vgc10.urdf.xacro (robot description, xacro)
@@ -12,4 +12,5 @@
     <xacro:include filename="$(find rbkairos_description)/urdf/structures/vgc10.urdf.xacro" />
     <xacro:include filename="$(find rbkairos_description)/urdf/structures/vgc10.gazebo.xacro" />
+    <xacro:include filename="$(find rbkairos_description)/urdf/structures/realsense2vgc10_support.urdf.xacro" />
   	<!-- Import summit XL wheels -->
   	<xacro:include filename="$(find summit_xl_description)/urdf/wheels/omni_wheel.urdf.xacro" />
@@ -153,4 +154,12 @@
   			<origin xyz="${right_holder_offset_x} ${right_holder_offset_y} ${right_holder_offset_z}" rpy="0 0 0"/>
   		</xacro:holder>
+        <!-- Intel Realsense support-->
+        <!--xacro:realsense2vgc10_support prefix="$(arg prefix)wrist_rgbd_support" parent="$(arg prefix)arm_tool0">
+            <origin xyz="0.0 0.0 0.0" rpy="0 0 0.0"/>
+  		</xacro:realsense2vgc10_support-->
+    	<!-- Intel Realsense -->
+    	<xacro:sensor_intel_d435 prefix="$(arg prefix)wrist_rgbd" parent="$(arg prefix)arm_tool0" prefix_topic="wrist_rgbd">
+      		<origin xyz="0.07 0.0 0.065" rpy="${pi} ${-pi/2} 0"/>
+    	</xacro:sensor_intel_d435>
 <gazebo>
   <plugin name="ground_truth_controller" filename="librobotnik_gazebo_ground_truth_odom.so">

Commit message: updated holder box model

File: rbkairos_description/robots/versions/rbkairos_ur5_oem_vgc10.urdf.xacro (robot description, xacro)
@@ -60,7 +60,7 @@
   	<xacro:property name="gps_offset_z" value="0.302"/>
 	<!-- Holder parameters -->
-  	<xacro:property name="centered_holder_offset_x" value="-0.195"/>
-  	<xacro:property name="centered_holder_offset_y" value="0.0"/>
-  	<xacro:property name="centered_holder_offset_z" value="0.56162"/>
+  	<xacro:property name="center_holder_offset_x" value="-0.195"/>
+  	<xacro:property name="center_holder_offset_y" value="0.0"/>
+  	<xacro:property name="center_holder_offset_z" value="0.56162"/>
   	<xacro:property name="left_holder_offset_x" value="-0.195"/>
   	<xacro:property name="left_holder_offset_y" value="0.225"/>
@@ -145,6 +145,6 @@
   		</xacro:sensor_zed-->
 		<!-- HOLDERS -->
-  		<xacro:holder prefix="${prefix}centered_" parent="${prefix}base_link">
-  			<origin xyz="${centered_holder_offset_x} ${centered_holder_offset_y} ${centered_holder_offset_z}" rpy="0 0 0"/>
+  		<xacro:holder prefix="${prefix}center_" parent="${prefix}base_link">
+  			<origin xyz="${center_holder_offset_x} ${center_holder_offset_y} ${center_holder_offset_z}" rpy="0 0 0"/>
   		</xacro:holder>
   		<xacro:holder prefix="${prefix}left_" parent="${prefix}base_link">
@@ -159,7 +159,7 @@
   		</xacro:realsense2vgc10_support-->
     	<!-- Intel Realsense -->
-    	<xacro:sensor_intel_d435 prefix="$(arg prefix)wrist_rgbd" parent="$(arg prefix)arm_tool0" prefix_topic="wrist_rgbd">
-      		<origin xyz="0.07 0.0 0.065" rpy="${pi} ${-pi/2} 0"/>
-    	</xacro:sensor_intel_d435>
+        <!--<xacro:sensor_intel_d435 prefix="$(arg prefix)wrist_rgbd" parent="$(arg prefix)arm_tool0" prefix_topic="wrist_rgbd">-->
+              <!--<origin xyz="0.07 0.0 0.065" rpy="${pi} ${-pi/2} 0"/>-->
+        <!--</xacro:sensor_intel_d435>-->
 <gazebo>
   <plugin name="ground_truth_controller" filename="librobotnik_gazebo_ground_truth_odom.so">

File: rbkairos_description/urdf/box/holder.urdf.xacro (robot description, xacro)
@@ -5,5 +5,5 @@
   <xacro:property name="prefix" value="$(arg prefix)" /-->
   <xacro:macro name="holder" params="prefix parent *origin">
-    <joint name="${prefix}holder2robot_joint" type="fixed">
+    <joint name="${prefix}holder_base_joint" type="fixed">
       <xacro:insert_block name="origin" />
       <parent link="${parent}"/>
@@ -13,5 +13,5 @@
     </link>
     <joint name="${prefix}holder_joint" type="fixed">
-      <origin rpy="1.57 0 0" xyz="0 0 0"/>
+      <origin rpy="0 0 0" xyz="0 0 0"/>
       <parent link="${prefix}holder_base_link"/>
       <child link="${prefix}holder_link"/>
@@ -36,4 +36,10 @@
       </collision>
     </link>
+    <joint name="${prefix}holder_approach_joint" type="fixed">
+      <origin rpy="3.1415 0 0" xyz="0 0 0.5"/>
+      <parent link="${prefix}holder_link"/>
+      <child link="${prefix}holder_approach_link"/>
+    </joint>
+    <link name="${prefix}holder_approach_link"/>
     <gazebo reference="${prefix}holder_link">
       <visual>
