Commit message: remove unused components

File: rbkairos_description/robots/versions/rbkairos_ur5_oem_vgc10.urdf.xacro (robot description, xacro)
@@ -1,28 +1,26 @@
 <?xml version="1.0"?>
 <robot name="rbkairos" xmlns:xacro="http://wiki.ros.org/xacro">
-  	<!-- ***************** -->
-  	<!-- Imported elements -->
-  	<!-- ***************** -->
-  	<!-- First we import all posible elements defined in the urdf.xacro files. All these elements are defined as macro:xacros -->
-  	<!-- Import summit XL base elements -->
-  	<xacro:include filename="$(find summit_xl_description)/urdf/bases/summit_xlsk_base_oem.urdf.xacro" />
+    <!-- ***************** -->
+    <!-- Imported elements -->
+    <!-- ***************** -->
+    <!-- First we import all posible elements defined in the urdf.xacro files. All these elements are defined as macro:xacros -->
+    <!-- Import summit XL base elements -->
+    <xacro:include filename="$(find summit_xl_description)/urdf/bases/summit_xlsk_base_oem.urdf.xacro" />
     <!-- Include UR-5 ARM -->
-	<xacro:include filename="$(find ur_description)/urdf/ur5.urdf.xacro" />
-	<!-- Include OnRobot vgc10 -->
+    <xacro:include filename="$(find ur_description)/urdf/ur5.urdf.xacro" />
+    <!-- Include OnRobot vgc10 -->
     <xacro:include filename="$(find rbkairos_description)/urdf/structures/vgc10.urdf.xacro" />
     <xacro:include filename="$(find rbkairos_description)/urdf/structures/vgc10.gazebo.xacro" />
     <xacro:include filename="$(find rbkairos_description)/urdf/structures/realsense2vgc10_support.urdf.xacro" />
-  	<!-- Import summit XL wheels -->
-  	<xacro:include filename="$(find summit_xl_description)/urdf/wheels/omni_wheel.urdf.xacro" />
-  	<xacro:include filename="$(find summit_xl_description)/urdf/wheels/rubber_wheel.urdf.xacro" />
-  	<xacro:include filename="$(find summit_xl_description)/urdf/structures/structure_hokuyo.urdf.xacro" />
-    <!-- Import holder for the boxes -->
-	<xacro:include filename="$(find rbkairos_description)/urdf/box/holder.urdf.xacro" />
-  	<!-- Import all available sensors -->
-  	<xacro:include filename="$(find robotnik_sensors)/urdf/all_sensors.urdf.xacro" />
-  	<xacro:property name="PI" value="3.1415926535897931"/>
+    <!-- Import summit XL wheels -->
+    <xacro:include filename="$(find summit_xl_description)/urdf/wheels/omni_wheel.urdf.xacro" />
+    <xacro:include filename="$(find summit_xl_description)/urdf/wheels/rubber_wheel.urdf.xacro" />
+    <xacro:include filename="$(find summit_xl_description)/urdf/structures/structure_hokuyo.urdf.xacro" />
+    <!-- Import all available sensors -->
+    <xacro:include filename="$(find robotnik_sensors)/urdf/all_sensors.urdf.xacro" />
+    <xacro:property name="PI" value="3.1415926535897931"/>
     <!-- Arguments set on rbkairos_state.launch -->
-  	<xacro:arg name="prefix" default="robot_"/>
-  	<xacro:arg name="ros_planar_move_plugin" default="false"/>
+    <xacro:arg name="prefix" default="robot_"/>
+    <xacro:arg name="ros_planar_move_plugin" default="false"/>
     <xacro:arg name="load_kinematics_file" default="false"/> <!-- Necesarry for ur_description compatible with official ur drivers-->
     <!-- Arm parameters -->
@@ -33,44 +31,34 @@
     <xacro:property name="arm_orientation_p" value="0"/>
     <xacro:property name="arm_orientation_y" value="0"/>
-  	<!-- Wheel parameters -->
-  	<xacro:property name="wheel_offset_x" value="0.21528" />    <!-- x,y,z in translation from base_link to the center of the wheel -->
-  	<xacro:property name="wheel_offset_y" value="0.2690" />
-  	<xacro:property name="wheel_offset_z" value="0.0" />
-  	<!-- Sensors parameters -->
-  	<xacro:property name="front_laser_offset_x" value="0.28783"/>
-  	<xacro:property name="front_laser_offset_y" value="-0.2224"/>
-  	<xacro:property name="front_laser_offset_z" value="0.30365"/>
-  	<xacro:property name="rear_laser_offset_x" value="-0.28783"/>
-  	<xacro:property name="rear_laser_offset_y" value="0.2224"/>
-  	<xacro:property name="rear_laser_offset_z" value="0.30365"/>
-  	<xacro:property name="front_ptz_camera_offset_x" value="0.308"/>
-  	<xacro:property name="front_ptz_camera_offset_y" value="0.141"/>
-  	<xacro:property name="front_ptz_camera_offset_z" value="0.195"/>
-  	<xacro:property name="rear_ptz_camera_offset_x" value="-0.308"/>
-  	<xacro:property name="rear_ptz_camera_offset_y" value="-0.141"/>
-  	<xacro:property name="rear_ptz_camera_offset_z" value="0.195"/>
+    <!-- Wheel parameters -->
+    <xacro:property name="wheel_offset_x" value="0.21528" />    <!-- x,y,z in translation from base_link to the center of the wheel -->
+    <xacro:property name="wheel_offset_y" value="0.2690" />
+    <xacro:property name="wheel_offset_z" value="0.0" />
+    <!-- Sensors parameters -->
+    <xacro:property name="front_laser_offset_x" value="0.28783"/>
+    <xacro:property name="front_laser_offset_y" value="-0.2224"/>
+    <xacro:property name="front_laser_offset_z" value="0.30365"/>
+    <xacro:property name="rear_laser_offset_x" value="-0.28783"/>
+    <xacro:property name="rear_laser_offset_y" value="0.2224"/>
+    <xacro:property name="rear_laser_offset_z" value="0.30365"/>
+    <xacro:property name="front_ptz_camera_offset_x" value="0.308"/>
+    <xacro:property name="front_ptz_camera_offset_y" value="0.141"/>
+    <xacro:property name="front_ptz_camera_offset_z" value="0.195"/>
+    <xacro:property name="rear_ptz_camera_offset_x" value="-0.308"/>
+    <xacro:property name="rear_ptz_camera_offset_y" value="-0.141"/>
+    <xacro:property name="rear_ptz_camera_offset_z" value="0.195"/>
     <xacro:property name="imu_offset_x" value="0.127"/>
-  	<xacro:property name="imu_offset_y" value="-0.129"/>
-  	<xacro:property name="imu_offset_z" value="0.212"/>
-  	<xacro:property name="front_rgbd_camera_offset_x" value="0.35850"/>
-  	<xacro:property name="front_rgbd_camera_offset_y" value="0.0"/>
-  	<xacro:property name="front_rgbd_camera_offset_z" value="0.25062"/>
-  	<xacro:property name="gps_offset_x" value="-0.365"/>
-  	<xacro:property name="gps_offset_y" value="-0.167"/>
-  	<xacro:property name="gps_offset_z" value="0.302"/>
-	<!-- Holder parameters -->
-  	<xacro:property name="center_holder_offset_x" value="-0.195"/>
-  	<xacro:property name="center_holder_offset_y" value="0.0"/>
-  	<xacro:property name="center_holder_offset_z" value="0.56162"/>
-  	<xacro:property name="left_holder_offset_x" value="-0.195"/>
-  	<xacro:property name="left_holder_offset_y" value="0.225"/>
-  	<xacro:property name="left_holder_offset_z" value="0.56162"/>
-  	<xacro:property name="right_holder_offset_x" value="-0.195"/>
-  	<xacro:property name="right_holder_offset_y" value="-0.225"/>
-  	<xacro:property name="right_holder_offset_z" value="0.56162"/>
-  	<!-- Flag to select the high or low quality model -->
-  	<xacro:property name="hq" value="true" />
-  	<xacro:arg name="prefix" default="robot_"/>
-  	<xacro:arg name="ros_planar_move_plugin" default="false"/>
+    <xacro:property name="imu_offset_y" value="-0.129"/>
+    <xacro:property name="imu_offset_z" value="0.212"/>
+    <xacro:property name="front_rgbd_camera_offset_x" value="0.35850"/>
+    <xacro:property name="front_rgbd_camera_offset_y" value="0.0"/>
+    <xacro:property name="front_rgbd_camera_offset_z" value="0.25062"/>
+    <xacro:property name="gps_offset_x" value="-0.365"/>
+    <xacro:property name="gps_offset_y" value="-0.167"/>
+    <xacro:property name="gps_offset_z" value="0.302"/>
+    <!-- Flag to select the high or low quality model -->
+    <xacro:property name="hq" value="true" />
+    <xacro:arg name="prefix" default="robot_"/>
+    <xacro:arg name="ros_planar_move_plugin" default="false"/>
     <xacro:arg name="load_kinematics_file" default="false"/> <!-- Necesarry for ur_description compatible with official ur drivers-->
     <xacro:property name="arm_position_x" value="0.15887"/>
@@ -81,24 +69,24 @@
     <xacro:property name="arm_orientation_y" value="0"/>
     <xacro:macro name="rbkairos" params="prefix publish_bf hq load_kinematics_file">
-  		<!-- *************** -->
-  		<!-- Robots Elements -->
-  		<!-- *************** -->
-  		<!-- Here we create the robot elements using the xacro:macros imported at the beggining of this file -->
-  		<!-- Summit XL base -->
-  		<xacro:summit_xls_base prefix="${prefix}" publish_bf="true" hq="${hq}" />
-  		<xacro:omni_wheel prefix="${prefix}front_right" parent="${prefix}base_link" reflect="false" hq="${hq}">
-  			<origin xyz="${wheel_offset_x} -${wheel_offset_y} ${wheel_offset_z}" rpy="0 0 0"/>
-  		</xacro:omni_wheel>
-  		<xacro:omni_wheel prefix="${prefix}front_left" parent="${prefix}base_link" reflect="true" hq="${hq}">
-  			<origin xyz="${wheel_offset_x} ${wheel_offset_y} ${wheel_offset_z}" rpy="0 0 0"/>
-  		</xacro:omni_wheel>
-  		<xacro:omni_wheel prefix="${prefix}back_left" parent="${prefix}base_link" reflect="true" hq="${hq}">
-  			<origin xyz="-${wheel_offset_x} ${wheel_offset_y} ${wheel_offset_z}" rpy="0 0 0"/>
-  		</xacro:omni_wheel>
-  		<xacro:omni_wheel prefix="${prefix}back_right" parent="${prefix}base_link" reflect="false" hq="${hq}">
-  			<origin xyz="-${wheel_offset_x} -${wheel_offset_y} ${wheel_offset_z}" rpy="0 0 0"/>
-  		</xacro:omni_wheel>
+        <!-- *************** -->
+        <!-- Robots Elements -->
+        <!-- *************** -->
+        <!-- Here we create the robot elements using the xacro:macros imported at the beggining of this file -->
+        <!-- Summit XL base -->
+        <xacro:summit_xls_base prefix="${prefix}" publish_bf="true" hq="${hq}" />
+        <xacro:omni_wheel prefix="${prefix}front_right" parent="${prefix}base_link" reflect="false" hq="${hq}">
+            <origin xyz="${wheel_offset_x} -${wheel_offset_y} ${wheel_offset_z}" rpy="0 0 0"/>
+        </xacro:omni_wheel>
+        <xacro:omni_wheel prefix="${prefix}front_left" parent="${prefix}base_link" reflect="true" hq="${hq}">
+            <origin xyz="${wheel_offset_x} ${wheel_offset_y} ${wheel_offset_z}" rpy="0 0 0"/>
+        </xacro:omni_wheel>
+        <xacro:omni_wheel prefix="${prefix}back_left" parent="${prefix}base_link" reflect="true" hq="${hq}">
+            <origin xyz="-${wheel_offset_x} ${wheel_offset_y} ${wheel_offset_z}" rpy="0 0 0"/>
+        </xacro:omni_wheel>
+        <xacro:omni_wheel prefix="${prefix}back_right" parent="${prefix}base_link" reflect="false" hq="${hq}">
+            <origin xyz="-${wheel_offset_x} -${wheel_offset_y} ${wheel_offset_z}" rpy="0 0 0"/>
+        </xacro:omni_wheel>
         <!-- UR-5 ARM -->
-		<xacro:if value="$(arg load_kinematics_file)">
+        <xacro:if value="$(arg load_kinematics_file)">
             <xacro:ur5_robot prefix="${prefix}arm_" joint_limited="true"
             shoulder_pan_lower_limit="${-pi}" shoulder_pan_upper_limit="${pi}"
@@ -111,6 +99,6 @@
                 <child link="${prefix}arm_base_link" />
             </joint>
-		</xacro:if>
-		<xacro:unless value="$(arg load_kinematics_file)">
+        </xacro:if>
+        <xacro:unless value="$(arg load_kinematics_file)">
             <xacro:ur5_robot prefix="${prefix}arm_" joint_limited="true"
             shoulder_pan_lower_limit="${-pi}" shoulder_pan_upper_limit="${pi}"
@@ -122,74 +110,64 @@
             <child link="${prefix}arm_base_link" />
             </joint>
-		</xacro:unless>
+        </xacro:unless>
         <!-- OnRobot VGC-10 -->
         <xacro:vgc10 prefix="${prefix}vgc10" parent="${prefix}arm_tool0">
-        	<origin xyz="0 0 0" rpy="0 -${PI/2.0} 0"/>
+            <origin xyz="0 0 0" rpy="0 -${PI/2.0} 0"/>
         </xacro:vgc10>
         <!-- IMU -->
-  		<xacro:sensor_imu_hector prefix="${prefix}imu" parent="${prefix}base_link">
-  			<origin xyz="${imu_offset_x} ${imu_offset_y} ${imu_offset_z}" rpy="0 0 0"/>
-  		</xacro:sensor_imu_hector>
-  		<!-- SENSORS -->
-  		<xacro:sensor_sick_s300 prefix="${prefix}front_laser" parent="${prefix}base_link" prefix_topic="front_laser">
-  			<origin xyz="${front_laser_offset_x} ${front_laser_offset_y} ${front_laser_offset_z}" rpy="0 ${-PI} ${3/4*PI}" />
-  		</xacro:sensor_sick_s300>
-  		<xacro:sensor_sick_s300 prefix="${prefix}rear_laser" parent="${prefix}base_link" prefix_topic="rear_laser">
-  			<origin xyz="${rear_laser_offset_x} ${rear_laser_offset_y} ${rear_laser_offset_z}" rpy="0 ${-PI} ${-1/4*PI}" />
-  		</xacro:sensor_sick_s300>
-  		<xacro:sensor_orbbec_astra prefix="${prefix}front_rgbd_camera" parent="${prefix}base_link" prefix_topic="front_rgbd_camera">
-  			<origin xyz="${front_rgbd_camera_offset_x} ${front_rgbd_camera_offset_y} ${front_rgbd_camera_offset_z}" rpy="0 0 0"/>
-  		</xacro:sensor_orbbec_astra>
-		<!--xacro:sensor_zed prefix="${prefix}front_rgbd_camera" parent="${prefix}base_link" prefix_topic="front_rgbd_camera">
-  			<origin xyz="${front_rgbd_camera_offset_x} ${front_rgbd_camera_offset_y} ${front_rgbd_camera_offset_z}" rpy="0 0 0"/>
-  		</xacro:sensor_zed-->
-		<!-- HOLDERS -->
-  		<xacro:holder prefix="${prefix}center_" parent="${prefix}base_link">
-  			<origin xyz="${center_holder_offset_x} ${center_holder_offset_y} ${center_holder_offset_z}" rpy="0 0 0"/>
-  		</xacro:holder>
-  		<xacro:holder prefix="${prefix}left_" parent="${prefix}base_link">
-  			<origin xyz="${left_holder_offset_x} ${left_holder_offset_y} ${left_holder_offset_z}" rpy="0 0 0"/>
-  		</xacro:holder>
-  		<xacro:holder prefix="${prefix}right_" parent="${prefix}base_link">
-  			<origin xyz="${right_holder_offset_x} ${right_holder_offset_y} ${right_holder_offset_z}" rpy="0 0 0"/>
-  		</xacro:holder>
+        <xacro:sensor_imu_hector prefix="${prefix}imu" parent="${prefix}base_link">
+            <origin xyz="${imu_offset_x} ${imu_offset_y} ${imu_offset_z}" rpy="0 0 0"/>
+        </xacro:sensor_imu_hector>
+        <!-- SENSORS -->
+        <xacro:sensor_sick_s300 prefix="${prefix}front_laser" parent="${prefix}base_link" prefix_topic="front_laser">
+            <origin xyz="${front_laser_offset_x} ${front_laser_offset_y} ${front_laser_offset_z}" rpy="0 ${-PI} ${3/4*PI}" />
+        </xacro:sensor_sick_s300>
+        <xacro:sensor_sick_s300 prefix="${prefix}rear_laser" parent="${prefix}base_link" prefix_topic="rear_laser">
+            <origin xyz="${rear_laser_offset_x} ${rear_laser_offset_y} ${rear_laser_offset_z}" rpy="0 ${-PI} ${-1/4*PI}" />
+        </xacro:sensor_sick_s300>
+        <xacro:sensor_orbbec_astra prefix="${prefix}front_rgbd_camera" parent="${prefix}base_link" prefix_topic="front_rgbd_camera">
+            <origin xyz="${front_rgbd_camera_offset_x} ${front_rgbd_camera_offset_y} ${front_rgbd_camera_offset_z}" rpy="0 0 0"/>
+        </xacro:sensor_orbbec_astra>
+        <!--xacro:sensor_zed prefix="${prefix}front_rgbd_camera" parent="${prefix}base_link" prefix_topic="front_rgbd_camera">
+            <origin xyz="${front_rgbd_camera_offset_x} ${front_rgbd_camera_offset_y} ${front_rgbd_camera_offset_z}" rpy="0 0 0"/>
+        </xacro:sensor_zed-->
         <!-- Intel Realsense support-->
         <!--xacro:realsense2vgc10_support prefix="$(arg prefix)wrist_rgbd_support" parent="$(arg prefix)arm_tool0">
             <origin xyz="0.0 0.0 0.0" rpy="0 0 0.0"/>
-  		</xacro:realsense2vgc10_support-->
-    	<!-- Intel Realsense -->
+        </xacro:realsense2vgc10_support-->
+        <!-- Intel Realsense -->
         <!--<xacro:sensor_intel_d435 prefix="$(arg prefix)wrist_rgbd" parent="$(arg prefix)arm_tool0" prefix_topic="wrist_rgbd">-->
               <!--<origin xyz="0.07 0.0 0.065" rpy="${pi} ${-pi/2} 0"/>-->
         <!--</xacro:sensor_intel_d435>-->
-<gazebo>
-  <plugin name="ground_truth_controller" filename="librobotnik_gazebo_ground_truth_odom.so">
-    <alwaysOn>true</alwaysOn>
-    <updateRate>50.0</updateRate>
-    <bodyName>${prefix}base_link</bodyName> <!-- robot body to track, in gazebo -->
-    <frameName>base_link_gt</frameName> <!-- frame name of robot body to be published in ros -->
-    <worldBodyName>world</worldBodyName> <!-- fixed body where body is tracked, in gazebo -->
-    <worldFrameName>odom</worldFrameName> <!-- frame name of fixed body to be published in ros -->
-    <topicName>odom_gt</topicName>
-    <gaussianNoise>0.01</gaussianNoise>
-    <xyzOffsets>0 0 0</xyzOffsets>
-    <rpyOffsets>0 0 0</rpyOffsets>
-    <broadcastTF>True</broadcastTF>
-  </plugin>
-</gazebo>
-<gazebo>
-  <plugin name="ground_lasertruth_controller_" filename="librobotnik_gazebo_ground_truth_odom.so">
-    <alwaysOn>true</alwaysOn>
-    <updateRate>50.0</updateRate>
-    <bodyName>${prefix}front_laser_link</bodyName> <!-- robot body to track, in gazebo -->
-    <frameName>laser_gt</frameName> <!-- frame name of robot body to be published in ros -->
-    <worldBodyName>world</worldBodyName> <!-- fixed body where body is tracked, in gazebo -->
-    <worldFrameName>odom</worldFrameName> <!-- frame name of fixed body to be published in ros -->
-    <topicName>laser_gt</topicName>
-    <gaussianNoise>0.01</gaussianNoise>
-    <xyzOffsets>0 0 0</xyzOffsets>
-    <rpyOffsets>0 0 0</rpyOffsets>
-    <broadcastTF>True</broadcastTF>
-  </plugin>
-</gazebo>
+      <gazebo>
+        <plugin name="ground_truth_controller" filename="librobotnik_gazebo_ground_truth_odom.so">
+          <alwaysOn>true</alwaysOn>
+          <updateRate>50.0</updateRate>
+          <bodyName>${prefix}base_link</bodyName> <!-- robot body to track, in gazebo -->
+          <frameName>${prefix}base_link_gt</frameName> <!-- frame name of robot body to be published in ros -->
+          <worldBodyName>world</worldBodyName> <!-- fixed body where body is tracked, in gazebo -->
+          <worldFrameName>${prefix}odom</worldFrameName> <!-- frame name of fixed body to be published in ros -->
+          <topicName>odom_gt</topicName>
+          <gaussianNoise>0.01</gaussianNoise>
+          <xyzOffsets>0 0 0</xyzOffsets>
+          <rpyOffsets>0 0 0</rpyOffsets>
+          <broadcastTF>True</broadcastTF>
+        </plugin>
+      </gazebo>
+      <gazebo>
+        <plugin name="ground_lasertruth_controller_" filename="librobotnik_gazebo_ground_truth_odom.so">
+          <alwaysOn>true</alwaysOn>
+          <updateRate>50.0</updateRate>
+          <bodyName>${prefix}front_laser_link</bodyName> <!-- robot body to track, in gazebo -->
+          <frameName>laser_gt</frameName> <!-- frame name of robot body to be published in ros -->
+          <worldBodyName>world</worldBodyName> <!-- fixed body where body is tracked, in gazebo -->
+          <worldFrameName>odom</worldFrameName> <!-- frame name of fixed body to be published in ros -->
+          <topicName>laser_gt</topicName>
+          <gaussianNoise>0.01</gaussianNoise>
+          <xyzOffsets>0 0 0</xyzOffsets>
+          <rpyOffsets>0 0 0</rpyOffsets>
+          <broadcastTF>True</broadcastTF>
+        </plugin>
+      </gazebo>
     </xacro:macro>
     <!-- Gazebo ros control pluggins -->
