Commit message: removed warning from moveit integration
non existent transforms (from gt plugin) and
non actuated joints (from gripper) which caused
invalid states

File: rbkairos_description/robots/versions/rbkairos_ur5_oem_vgc10.urdf.xacro (robot description, xacro)
@@ -140,34 +140,34 @@
               <origin xyz="0.07 0.0 0.065" rpy="${pi} ${-pi/2} 0"/>
         </xacro:sensor_intel_d435>
-      <gazebo>
-        <plugin name="ground_truth_controller" filename="librobotnik_gazebo_ground_truth_odom.so">
-          <alwaysOn>true</alwaysOn>
-          <updateRate>50.0</updateRate>
-          <bodyName>${prefix}base_link</bodyName> <!-- robot body to track, in gazebo -->
-          <frameName>${prefix}base_link_gt</frameName> <!-- frame name of robot body to be published in ros -->
-          <worldBodyName>world</worldBodyName> <!-- fixed body where body is tracked, in gazebo -->
-          <worldFrameName>${prefix}odom</worldFrameName> <!-- frame name of fixed body to be published in ros -->
-          <topicName>odom_gt</topicName>
-          <gaussianNoise>0.01</gaussianNoise>
-          <xyzOffsets>0 0 0</xyzOffsets>
-          <rpyOffsets>0 0 0</rpyOffsets>
-          <broadcastTF>True</broadcastTF>
-        </plugin>
-      </gazebo>
-      <gazebo>
-        <plugin name="ground_lasertruth_controller_" filename="librobotnik_gazebo_ground_truth_odom.so">
-          <alwaysOn>true</alwaysOn>
-          <updateRate>50.0</updateRate>
-          <bodyName>${prefix}front_laser_link</bodyName> <!-- robot body to track, in gazebo -->
-          <frameName>laser_gt</frameName> <!-- frame name of robot body to be published in ros -->
-          <worldBodyName>world</worldBodyName> <!-- fixed body where body is tracked, in gazebo -->
-          <worldFrameName>odom</worldFrameName> <!-- frame name of fixed body to be published in ros -->
-          <topicName>laser_gt</topicName>
-          <gaussianNoise>0.01</gaussianNoise>
-          <xyzOffsets>0 0 0</xyzOffsets>
-          <rpyOffsets>0 0 0</rpyOffsets>
-          <broadcastTF>True</broadcastTF>
-        </plugin>
-      </gazebo>
+      <!--<gazebo>-->
+        <!--<plugin name="ground_truth_controller" filename="librobotnik_gazebo_ground_truth_odom.so">-->
+          <!--<alwaysOn>true</alwaysOn>-->
+          <!--<updateRate>50.0</updateRate>-->
+          <!--<bodyName>${prefix}base_link</bodyName> [> robot body to track, in gazebo <]-->
+          <!--<frameName>${prefix}base_link_gt</frameName> [> frame name of robot body to be published in ros <]-->
+          <!--<worldBodyName>world</worldBodyName> [> fixed body where body is tracked, in gazebo <]-->
+          <!--<worldFrameName>${prefix}odom</worldFrameName> [> frame name of fixed body to be published in ros <]-->
+          <!--<topicName>odom_gt</topicName>-->
+          <!--<gaussianNoise>0.01</gaussianNoise>-->
+          <!--<xyzOffsets>0 0 0</xyzOffsets>-->
+          <!--<rpyOffsets>0 0 0</rpyOffsets>-->
+          <!--<broadcastTF>True</broadcastTF>-->
+        <!--</plugin>-->
+      <!--</gazebo>-->
+      <!--<gazebo>-->
+        <!--<plugin name="ground_lasertruth_controller_" filename="librobotnik_gazebo_ground_truth_odom.so">-->
+          <!--<alwaysOn>true</alwaysOn>-->
+          <!--<updateRate>50.0</updateRate>-->
+          <!--<bodyName>${prefix}front_laser_link</bodyName> [> robot body to track, in gazebo <]-->
+          <!--<frameName>laser_gt</frameName> [> frame name of robot body to be published in ros <]-->
+          <!--<worldBodyName>world</worldBodyName> [> fixed body where body is tracked, in gazebo <]-->
+          <!--<worldFrameName>odom</worldFrameName> [> frame name of fixed body to be published in ros <]-->
+          <!--<topicName>laser_gt</topicName>-->
+          <!--<gaussianNoise>0.01</gaussianNoise>-->
+          <!--<xyzOffsets>0 0 0</xyzOffsets>-->
+          <!--<rpyOffsets>0 0 0</rpyOffsets>-->
+          <!--<broadcastTF>True</broadcastTF>-->
+        <!--</plugin>-->
+      <!--</gazebo>-->
     <!-- Gazebo ros control pluggins -->
     <xacro:ros_control/>

File: rbkairos_description/urdf/structures/vgc10.urdf.xacro (robot description, xacro)
@@ -36,5 +36,5 @@
       <child link="${prefix}_vacuum_cup_1_link"/>
       <axis xyz="1 0 0" rpy="0 0 0" />
-      <limit effort="30" velocity="1.0" lower="0" upper="0" />
+      <limit effort="30" velocity="1.0" lower="-0.1" upper="0.1" />
     </joint>
     <link name="${prefix}_vacuum_cup_1_link">
@@ -50,5 +50,5 @@
       <child link="${prefix}_vacuum_cup_2_link"/>
       <axis xyz="1 0 0" rpy="0 0 0" />
-      <limit effort="30" velocity="1.0" lower="0" upper="0" />
+      <limit effort="30" velocity="1.0" lower="-0.1" upper="0.1" />
     </joint>
     <link name="${prefix}_vacuum_cup_2_link">
@@ -63,5 +63,5 @@
       <parent link="${prefix}_vgc10_link"/>
       <child link="${prefix}_vacuum_cup_3_link"/>
-      <limit effort="30" velocity="1.0" lower="0" upper="0" />
+      <limit effort="30" velocity="1.0" lower="-0.1" upper="0.1" />
       <axis xyz="1 0 0" rpy="0 0 0" />
     </joint>
@@ -77,5 +77,5 @@
       <parent link="${prefix}_vgc10_link"/>
       <child link="${prefix}_vacuum_cup_4_link"/>
-      <limit effort="30" velocity="1.0" lower="0" upper="0" />
+      <limit effort="30" velocity="1.0" lower="-0.1" upper="0.1" />
       <axis xyz="1 0 0" rpy="0 0 0" />
     </joint>
