Commit message: Add MoveIt config for ur5 arm with egh gripper

File: rbkairos_description/robots/versions/rbkairos_ur5_egh.urdf.xacro (robot description, xacro)
@@ -60,6 +60,6 @@
 		</xacro:egh_gripper>
         <!-- Intel Realsense -->
-    <xacro:sensor_r430 prefix="$(arg prefix)arm_rgbd_camera" parent="$(arg prefix)arm_tool0" prefix_topic="front_rgbd_camera">
-      <origin xyz="0.0 -0.05 -0.01" rpy="${pi/2} ${-pi/2} 0"/>
+    <xacro:sensor_r430 prefix="$(arg prefix)wrist_rgbd" parent="$(arg prefix)arm_tool0" prefix_topic="wrist_rgbd">
+      <origin xyz="-0.075 0.0 0.065" rpy="0 ${-pi/2} 0"/>
     </xacro:sensor_r430>
 	</xacro:macro>

Commit message: rbkairos_description: update arm orientation

File: rbkairos_description/robots/versions/rbkairos_ur5_egh.urdf.xacro (robot description, xacro)
@@ -23,5 +23,5 @@
   <xacro:property name="arm_orientation_r" value="0"/>
   <xacro:property name="arm_orientation_p" value="0"/>
-  <xacro:property name="arm_orientation_y" value="${-3*pi/4}"/>
+  <xacro:property name="arm_orientation_y" value="${3*pi/4}"/>
   <xacro:macro name="rbkairos" params="prefix publish_bf hq load_kinematics_file">
 		<!-- *************** -->

Commit message: Updates rbkairos_ur5_egh to use new files from UR repo

File: rbkairos_description/robots/versions/rbkairos_ur5_egh.urdf.xacro (robot description, xacro)
@@ -8,5 +8,5 @@
 	<xacro:include filename="$(find rbkairos_description)/urdf/bases/rbkairos_base.urdf.xacro" />
 	<!-- Include UR-5 ARM -->
-	<xacro:include filename="$(find ur_description)/urdf/ur5.urdf.xacro" />
+	<xacro:include filename="$(find ur_description)/urdf/inc/ur5_macro.xacro" />
   <!-- Include EGH TODO -->
 	<xacro:include filename="$(find egh_gripper_description)/urdf/egh_gripper.urdf.xacro" />
@@ -32,27 +32,11 @@
 		<xacro:rbkairos_base prefix="$(arg prefix)" publish_bf="true" hq="true"/>
 		<!-- UR-5 ARM -->
-		<xacro:if value="$(arg load_kinematics_file)">
-        <xacro:ur5_robot prefix="$(arg prefix)arm_" joint_limited="true"
-          shoulder_pan_lower_limit="${-pi}" shoulder_pan_upper_limit="${pi}"
-          wrist_3_lower_limit="${-pi}" wrist_3_upper_limit="${pi}"
-          kinematics_file="${load_yaml('$(find rbkairos_control)/config/ur5_calibration.yaml')}">
-        </xacro:ur5_robot>
-        <joint name="$(arg prefix)arm_base_joint" type="fixed">
-          <origin xyz="${arm_position_x} ${arm_position_y} ${arm_position_z}" rpy="${arm_orientation_r} ${arm_orientation_p} ${arm_orientation_y}"/>
-          <parent link="$(arg prefix)base_link" />
-          <child link="$(arg prefix)arm_base_link" />
-        </joint>
-		</xacro:if>
-		<xacro:unless value="$(arg load_kinematics_file)">
-        <xacro:ur5_robot prefix="$(arg prefix)arm_" joint_limited="true"
-          shoulder_pan_lower_limit="${-pi}" shoulder_pan_upper_limit="${pi}"
-          wrist_3_lower_limit="${-pi}" wrist_3_upper_limit="${pi}">
-        </xacro:ur5_robot>
-        <joint name="$(arg prefix)arm_base_joint" type="fixed">
-          <origin xyz="${arm_position_x} ${arm_position_y} ${arm_position_z}" rpy="${arm_orientation_r} ${arm_orientation_p} ${arm_orientation_y}"/>
-          <parent link="$(arg prefix)base_link" />
-          <child link="$(arg prefix)arm_base_link" />
-        </joint>
-		</xacro:unless>
+    <xacro:ur5_robot prefix="$(arg prefix)arm_" >
+    </xacro:ur5_robot>
+    <joint name="$(arg prefix)arm_base_joint" type="fixed">
+      <origin xyz="${arm_position_x} ${arm_position_y} ${arm_position_z}" rpy="${arm_orientation_r} ${arm_orientation_p} ${arm_orientation_y}"/>
+      <parent link="$(arg prefix)base_link" />
+      <child link="$(arg prefix)arm_base_link" />
+    </joint>
 		<!-- Schunk EGH -->
 		<xacro:egh_gripper prefix="$(arg prefix)egh_gripper" parent="$(arg prefix)arm_tool0">
@@ -69,4 +53,4 @@
    </xacro:if>
 	</xacro:macro>
-   <!--xacro:rbkairos_ur10_wsg50 prefix="$(arg prefix)" publish_bf="true" hq="true" load_kinematics_file="$(arg load_kinematics_file)"/-->
+   <xacro:rbkairos_ur5_egh prefix="$(arg prefix)" publish_bf="true" hq="true" load_kinematics_file="$(arg load_kinematics_file)"/>
 </robot>
