Commit message: Corrected issue with names and inertias

File: rbkairos_description/urdf/structures/vgc10.gazebo.xacro (robot description, xacro)
@@ -6,6 +6,6 @@
        <robotNamespace>/robot</robotNamespace>
        <bodyName>robot_vgc10_vacuum_cup_1_link</bodyName>
-       <topicName>grasping_cup_1</topicName>
-       <serviceNamespace>gripper_1</serviceNamespace>
+       <topicName>vacuum_cup_1</topicName>
+       <serviceNamespace>vacuum_cup_1</serviceNamespace>
      </plugin>
    </gazebo>

File: rbkairos_description/urdf/structures/vgc10.urdf.xacro (robot description, xacro)
@@ -38,5 +38,11 @@
       <limit effort="30" velocity="1.0" lower="0" upper="0" />
     </joint>
-    <link name="${prefix}_vacuum_cup_1_link"/>
+    <link name="${prefix}_vacuum_cup_1_link">
+      <inertial>
+        <origin xyz="0 0 0" rpy="0 0 0"/>
+        <mass value="0.01"/>
+        <inertia ixx="0.000001"  ixy="0"  ixz="0" iyy="0.000001" iyz="0" izz="0.000001" />
+      </inertial>
+    </link>
     <joint name="${prefix}_vacuum_cup_2_joint" type="revolute">
       <origin xyz="0.1322 -0.0065 0.0189" rpy="0 0 0"/>
@@ -46,5 +52,11 @@
       <limit effort="30" velocity="1.0" lower="0" upper="0" />
     </joint>
-    <link name="${prefix}_vacuum_cup_2_link"/>
+    <link name="${prefix}_vacuum_cup_2_link">
+      <inertial>
+        <origin xyz="0 0 0" rpy="0 0 0"/>
+        <mass value="0.01"/>
+        <inertia ixx="0.000001"  ixy="0"  ixz="0" iyy="0.000001" iyz="0" izz="0.000001" />
+      </inertial>
+    </link>
     <joint name="${prefix}_vacuum_cup_3_joint" type="revolute">
       <origin xyz="0.1322 0.02 0" rpy="0 0 0"/>
@@ -54,5 +66,11 @@
       <axis xyz="1 0 0" rpy="0 0 0" />
     </joint>
-    <link name="${prefix}_vacuum_cup_3_link"/>
+    <link name="${prefix}_vacuum_cup_3_link">
+      <inertial>
+        <origin xyz="0 0 0" rpy="0 0 0"/>
+        <mass value="0.01"/>
+        <inertia ixx="0.000001"  ixy="0"  ixz="0" iyy="0.000001" iyz="0" izz="0.000001" />
+      </inertial>
+    </link>
     <joint name="${prefix}_vacuum_cup_4_joint" type="revolute">
       <origin xyz="0.1322 0 0" rpy="0 0 0"/>
@@ -62,42 +80,48 @@
       <axis xyz="1 0 0" rpy="0 0 0" />
     </joint>
-    <link name="${prefix}_vacuum_cup_4_link"/>
+    <link name="${prefix}_vacuum_cup_4_link">
+      <inertial>
+        <origin xyz="0 0 0" rpy="0 0 0"/>
+        <mass value="0.01"/>
+        <inertia ixx="0.000001"  ixy="0"  ixz="0" iyy="0.000001" iyz="0" izz="0.000001" />
+      </inertial>
+    </link>
     <!-- Transmission -->
-    <transmission name="${prefix}_vacuum_cup_1_joint">
+    <transmission name="${prefix}_vacuum_cup_1_joint_transmission">
       <type>transmission_interface/SimpleTransmission</type>
       <joint name="${prefix}_vacuum_cup_1_joint">
         <hardwareInterface>hardware_interface/PositionJointInterface</hardwareInterface>
       </joint>
-      <actuator name="${prefix}_vacuum_cup_1_joint">
+      <actuator name="${prefix}_vacuum_cup_1_joint_motor">
         <hardwareInterface>hardware_interface/PositionActuatorInterface</hardwareInterface>
         <mechanicalReduction>1</mechanicalReduction>
       </actuator>
     </transmission>
-    <transmission name="${prefix}_vacuum_cup_2_joint">
+    <transmission name="${prefix}_vacuum_cup_2_joint_transmission">
       <type>transmission_interface/SimpleTransmission</type>
       <joint name="${prefix}_vacuum_cup_2_joint">
         <hardwareInterface>hardware_interface/PositionJointInterface</hardwareInterface>
       </joint>
-      <actuator name="${prefix}_vacuum_cup_2_joint">
+      <actuator name="${prefix}_vacuum_cup_2_joint_motor">
         <hardwareInterface>hardware_interface/PositionActuatorInterface</hardwareInterface>
         <mechanicalReduction>1</mechanicalReduction>
       </actuator>
     </transmission>
-    <transmission name="${prefix}_vacuum_cup_3_joint">
+    <transmission name="${prefix}_vacuum_cup_3_joint_transmission">
       <type>transmission_interface/SimpleTransmission</type>
       <joint name="${prefix}_vacuum_cup_3_joint">
         <hardwareInterface>hardware_interface/PositionJointInterface</hardwareInterface>
       </joint>
-      <actuator name="${prefix}_vacuum_cup_3_joint">
+      <actuator name="${prefix}_vacuum_cup_3_joint_motor">
         <hardwareInterface>hardware_interface/PositionActuatorInterface</hardwareInterface>
         <mechanicalReduction>1</mechanicalReduction>
       </actuator>
     </transmission>
-    <transmission name="${prefix}_vacuum_cup_4_joint">
+    <transmission name="${prefix}_vacuum_cup_4_joint_transmission">
       <type>transmission_interface/SimpleTransmission</type>
       <joint name="${prefix}_vacuum_cup_4_joint">
         <hardwareInterface>hardware_interface/PositionJointInterface</hardwareInterface>
       </joint>
-      <actuator name="${prefix}_vacuum_cup_4_joint">
+      <actuator name="${prefix}_vacuum_cup_4_joint_motor">
         <hardwareInterface>hardware_interface/PositionActuatorInterface</hardwareInterface>
         <mechanicalReduction>1</mechanicalReduction>
