Commit message: Corrected vgc_10 urdf

File: rbkairos_description/urdf/structures/vgc10.urdf.xacro (robot description, xacro)
@@ -38,4 +38,30 @@
       <limit effort="30" velocity="1.0" lower="0" upper="0" />
     </joint>
+    <link name="${prefix}_vacuum_cup_1_link"/>
+    <joint name="${prefix}_vacuum_cup_2_joint" type="revolute">
+      <origin xyz="0.1322 -0.0065 0.0189" rpy="0 0 0"/>
+      <parent link="${prefix}_vgc10_link"/>
+      <child link="${prefix}_vacuum_cup_2_link"/>
+      <axis xyz="1 0 0" rpy="0 0 0" />
+      <limit effort="30" velocity="1.0" lower="0" upper="0" />
+    </joint>
+    <link name="${prefix}_vacuum_cup_2_link"/>
+    <joint name="${prefix}_vacuum_cup_3_joint" type="revolute">
+      <origin xyz="0.1322 0.02 0" rpy="0 0 0"/>
+      <parent link="${prefix}_vgc10_link"/>
+      <child link="${prefix}_vacuum_cup_3_link"/>
+      <limit effort="30" velocity="1.0" lower="0" upper="0" />
+      <axis xyz="1 0 0" rpy="0 0 0" />
+    </joint>
+    <link name="${prefix}_vacuum_cup_3_link"/>
+    <joint name="${prefix}_vacuum_cup_4_joint" type="revolute">
+      <origin xyz="0.1322 0 0" rpy="0 0 0"/>
+      <parent link="${prefix}_vgc10_link"/>
+      <child link="${prefix}_vacuum_cup_4_link"/>
+      <limit effort="30" velocity="1.0" lower="0" upper="0" />
+      <axis xyz="1 0 0" rpy="0 0 0" />
+    </joint>
+    <link name="${prefix}_vacuum_cup_4_link"/>
+    <!-- Transmission -->
     <transmission name="${prefix}_vacuum_cup_1_joint">
       <type>transmission_interface/SimpleTransmission</type>
@@ -48,12 +74,4 @@
       </actuator>
     </transmission>
-    <link name="${prefix}_vacuum_cup_1_link"/>
-    <joint name="${prefix}_vacuum_cup_2_joint" type="revolute">
-      <origin xyz="0.1322 -0.0065 0.0189" rpy="0 0 0"/>
-      <parent link="${prefix}_vgc10_link"/>
-      <child link="${prefix}_vacuum_cup_2_link"/>
-      <axis xyz="1 0 0" rpy="0 0 0" />
-      <limit effort="30" velocity="1.0" lower="0" upper="0" />
-    </joint>
     <transmission name="${prefix}_vacuum_cup_2_joint">
       <type>transmission_interface/SimpleTransmission</type>
@@ -66,12 +84,4 @@
       </actuator>
     </transmission>
-    <link name="${prefix}_vacuum_cup_2_link"/>
-    <joint name="${prefix}_vacuum_cup_3_joint" type="revolute">
-      <origin xyz="0.1322 0.02 0" rpy="0 0 0"/>
-      <parent link="${prefix}_vgc10_link"/>
-      <child link="${prefix}_vacuum_cup_3_link"/>
-      <limit effort="30" velocity="1.0" lower="0" upper="0" />
-      <axis xyz="1 0 0" rpy="0 0 0" />
-    </joint>
     <transmission name="${prefix}_vacuum_cup_3_joint">
       <type>transmission_interface/SimpleTransmission</type>
@@ -84,23 +94,14 @@
       </actuator>
     </transmission>
-    <link name="${prefix}_vacuum_cup_3_link"/>
-  <joint name="${prefix}_vacuum_cup_4_joint" type="revolute">
-    <origin xyz="0.1322 0 0" rpy="0 0 0"/>
-    <parent link="${prefix}_vgc10_link"/>
-    <child link="${prefix}_vacuum_cup_4_link"/>
-    <limit effort="30" velocity="1.0" lower="0" upper="0" />
-    <axis xyz="1 0 0" rpy="0 0 0" />
-  </joint>
-  <transmission name="${prefix}_vacuum_cup_4_joint">
-    <type>transmission_interface/SimpleTransmission</type>
-    <joint name="${prefix}_vacuum_cup_4_joint">
-      <hardwareInterface>hardware_interface/PositionJointInterface</hardwareInterface>
-    </joint>
-    <actuator name="${prefix}_vacuum_cup_4_joint">
-      <hardwareInterface>hardware_interface/PositionActuatorInterface</hardwareInterface>
-      <mechanicalReduction>1</mechanicalReduction>
-    </actuator>
-  </transmission>
-  <link name="${prefix}_vacuum_cup_4_link"/>
+    <transmission name="${prefix}_vacuum_cup_4_joint">
+      <type>transmission_interface/SimpleTransmission</type>
+      <joint name="${prefix}_vacuum_cup_4_joint">
+        <hardwareInterface>hardware_interface/PositionJointInterface</hardwareInterface>
+      </joint>
+      <actuator name="${prefix}_vacuum_cup_4_joint">
+        <hardwareInterface>hardware_interface/PositionActuatorInterface</hardwareInterface>
+        <mechanicalReduction>1</mechanicalReduction>
+      </actuator>
+    </transmission>
   </xacro:macro>
 </robot>

Commit message: rbkairos_description: Added simplified mesh for onrobot vgc10 gripper's collision tag, reduces MoveIt's loading time during initialization.

File: rbkairos_description/urdf/structures/vgc10.urdf.xacro (robot description, xacro)
@@ -27,5 +27,5 @@
 	      <geometry>
           <!--box size="0.12 0.1 0.1" /-->
-	        <mesh filename="package://rbkairos_description/meshes/structures/vgc10.stl"/>
+	        <mesh filename="package://rbkairos_description/meshes/structures/vgc10.dae"/>
 	      </geometry>
 	    </collision>
