Commit message: box.urdf.xacro: added grey color

File: rbkairos_description/urdf/box/box.urdf.xacro (robot description, xacro)
@@ -60,3 +60,23 @@
   </joint>
   <link name="${prefix}grasping_link"/>
+      <gazebo reference="${prefix}body_box_link">
+      <visual>
+        <material>
+          <ambient>0.0 0.0 0.0 1.0</ambient>
+          <diffuse>0.2 0.2 0.2 1.0</diffuse>
+          <specular>0.584313725 0.647058824 0.650980392 1.0</specular>
+          <emissive>0.0 0.0 0.0 0.0</emissive>
+        </material>
+      </visual>
+    </gazebo>
+      <gazebo reference="${prefix}handle_link">
+      <visual>
+        <material>
+          <ambient>0.0 0.0 0.0 1.0</ambient>
+          <diffuse>0.2 0.2 0.2 1.0</diffuse>
+          <specular>0.584313725 0.647058824 0.650980392 1.0</specular>
+          <emissive>0.0 0.0 0.0 0.0</emissive>
+        </material>
+      </visual>
+    </gazebo>
 </robot>
